File: Moog_Prodigy_Project/moog_prodigy_project/Schematics/Right_side.kicad_sch (KiCad schematic)
At the start: 0 parts

Commit message: Potrebno je da se uradi jos zamena za 4007, dal ubaciti pojedinacne mosfete ili ima vec neko integrisano kolo koje je slicno tome, koje parametre gledati
Other:
- added sheet 3046 (ledder.kicad_sch)
- added sheet 4007 (4007_mosfets.kicad_sch)
- added sheet dual_timer (dual_timer.kicad_sch)
- added sheet ledder (ledder_transistors.kicad_sch)
- added sheet vca_attack (vca_attack.kicad_sch)
- added sheet voltage_source (voltage_source.kicad_sch)
