File: Moog_Prodigy_Project/moog_prodigy_project/Schematics/ledder.kicad_sch (KiCad schematic)
At the start: 36 parts, among them Q100 CA3046, Q101 CA3046, Q102 BC556, Q103 BC556, U100 OPA184, U101 3080, U102 OPA184

Commit message: LT1227 added
Parts:
- U101: value 3080 -> LT1228
Connections:
- net enter_CP102: now reaches CP102.2
Changed lines of the file:
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@@
 	(wire
 		(pts
+			(xy 48.26 109.22) (xy 48.26 106.68)
+		)
+		(stroke
+			(width 0)
+			(type default)
+		)
+	)
+	(wire
+		(pts
 			(xy 83.82 62.23) (xy 83.82 72.39)
 		)
@@
 		)
 	)
+	(global_label "enter_CP102"
+		(shape input)
+		(at 48.26 109.22 270)
+		(fields_autoplaced yes)
+		(effects
+			(font
+				(size 1.27 1.27)
+			)
+			(justify right)
+		)
+		(property "Intersheetrefs" "${INTERSHEET_REFS}"
+			(at 48.26 124.1794 90)
+			(effects
+				(font
+					(size 1.27 1.27)
+				)
+				(justify right)
+				(hide yes)
+			)
+		)
+	)
 	(global_label "node_2"
 		(shape input)
@@
 			)
 		)
-		(property "Value" "3080"
+		(property "Value" "LT1228"
 			(at 226.822 93.472 0)
 			(effects

Commit message: Dodato zamena za 4007, bolje karakteristike po pitanju brzine samih fetova, nebaferovani (UB) zato sto nam treba linearna komponenta
Connections:
- net OUTPUT_2 renamed THRESHOLD_1
Changed lines of the file:
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@@
-		)
-	)
-	(global_label "OUTPUT_2"
-		(shape output)
-		(at 232.41 132.08 0)
-		(fields_autoplaced yes)
-		(effects
-			(font
-				(size 1.27 1.27)
-			)
-			(justify left)
-		)
-		(property "Intersheetrefs" "${INTERSHEET_REFS}"
-			(at 244.769 132.08 0)
-			(effects
-				(font
-					(size 1.27 1.27)
-				)
-				(justify left)
-				(hide yes)
-			)
 		)
 	)
@@
 				(hide yes)
 			)
+		)
+	)
+	(global_label "THRESHOLD_1"
+		(shape input)
+		(at 232.41 132.08 0)
+		(fields_autoplaced yes)
+		(effects
+			(font
+				(size 1.27 1.27)
+			)
+			(justify left)
+		)
+		(property "Intersheetrefs" "${INTERSHEET_REFS}"
+			(at 248.458 132.08 0)
+			(effects
+				(font
+					(size 1.27 1.27)
+				)
+				(justify left)
+				(hide yes)
+			)
