File: Moog_Prodigy_Project/moog_prodigy_project/Schematics/dual_timer.kicad_sch (KiCad schematic)
At the start: 3 parts, among them U3 NE556N

Commit message: transformator i prekidac
Parts:
- R100: footprint (none) -> Resistor_THT:R_Axial_DIN0207_L6.3mm_D2.5mm_P7.62mm_Horizontal
Changed lines of the file:
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@@
 			)
 		)
-		(property "Footprint" ""
+		(property "Footprint" "Resistor_THT:R_Axial_DIN0207_L6.3mm_D2.5mm_P7.62mm_Horizontal"
 			(at 151.892 54.61 90)
 			(effects
