File: Moog_Prodigy_Project/moog_prodigy_project/Schematics/vca_attack.kicad_sch (KiCad schematic)
At the start: 0 parts

Commit message: Dodato zamena za 4007, bolje karakteristike po pitanju brzine samih fetova, nebaferovani (UB) zato sto nam treba linearna komponenta
Parts:
- added C110, C111: 10n, symbol Device:C_Small
- added R143, R144, R149: 10K, symbol Device:R
- added R145, R146: 1K, symbol Device:R
- added R147: 1M, symbol Device:R
- added R148: 100k, symbol Device:R
- added RV113, RV114: 1M, symbol Device:R_Potentiometer
- added U105, U106, U107: MC14007UBCP, symbol MC14007UBCP:MC14007UBCP
Connections:
- new net: R149.1, U107.1
- new net: C111.1, R146.2, U107.3
- new net: R145.2, U107.10, U107.5
- new net: R145.1, U105.10, U106.10, U107.13, U107.8
- new net: C110.1, R147.2, U107.6
- new net: R144.1, U106.3, U106.8
- new net: RV114.3, U106.1
- new net: RV113.3, U105.1
- new net: R143.1, U105.3, U105.8
- new net: R147.1, R148.2
- new net +12V: R143.2, R144.2, U105.14, U105.2, U106.14, U106.2, U107.11, U107.14, U107.2
- new net GND: R146.1, R148.1, R149.2, U105.7, U105.9, U106.7, U106.9, U107.4, U107.7, U107.9
- new net OUTPUT_1: U105.6
- new net OUTPUT_2: U106.6
- new net RESET: C110.2, C111.2, U107.12
- new net VCA_ATTACK_PIN_12: U105.12
- new net VCF_ATTACK_PIN_12: U106.12
- new net node_10: U105.4
- new net node_11: RV114.1, RV114.2
- new net node_12: U106.5
- new net node_13: U106.4
- new net node_8: RV113.1, RV113.2
- new net node_9: U105.5
- no-connect marks 0 -> 4
Other:
- note added: "VCA ATTACK"
- note added: "VCF ATTACK"

Commit message: transformator i prekidac
Parts:
- C110, C111: footprint (none) -> Capacitor_THT:C_Disc_D3.8mm_W2.6mm_P2.50mm
- R143, R144, R145, R146, R147, R148, R149: footprint (none) -> Resistor_THT:R_Axial_DIN0207_L6.3mm_D2.5mm_P7.62mm_Horizontal
- RV113, RV114: footprint (none) -> Potentiometer_THT:Potentiometer_ACP_CA9-V10_Vertical
- U105, U106, U107: footprint (none) -> Package_DIP:DIP-14_W7.62mm_Socket
Changed lines of the file:
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@@
 			)
 		)
-		(property "Footprint" ""
+		(property "Footprint" "Resistor_THT:R_Axial_DIN0207_L6.3mm_D2.5mm_P7.62mm_Horizontal"
 			(at 133.35 114.808 90)
 			(effects
@@
 			)
 		)
-		(property "Footprint" ""
+		(property "Footprint" "Resistor_THT:R_Axial_DIN0207_L6.3mm_D2.5mm_P7.62mm_Horizontal"
 			(at 138.43 154.178 90)
 			(effects
@@
 			)
 		)
-		(property "Footprint" ""
+		(property "Footprint" "Package_DIP:DIP-14_W7.62mm_Socket"
 			(at 109.22 135.89 0)
 			(effects
@@
 			)
 		)
-		(property "Footprint" ""
+		(property "Footprint" "Resistor_THT:R_Axial_DIN0207_L6.3mm_D2.5mm_P7.62mm_Horizontal"
 			(at 116.84 154.178 90)
 			(effects
@@
 			)
 		)
-		(property "Footprint" ""
+		(property "Footprint" "Resistor_THT:R_Axial_DIN0207_L6.3mm_D2.5mm_P7.62mm_Horizontal"
 			(at 158.75 44.958 90)
 			(effects
@@
 			)
 		)
-		(property "Footprint" ""
+		(property "Footprint" "Potentiometer_THT:Potentiometer_ACP_CA9-V10_Vertical"
 			(at 180.34 43.18 0)
 			(effects
@@
 			)
 		)
-		(property "Footprint" ""
+		(property "Footprint" "Package_DIP:DIP-14_W7.62mm_Socket"
 			(at 67.31 73.66 0)
 			(effects
@@
 			)
 		)
-		(property "Footprint" ""
+		(property "Footprint" "Resistor_THT:R_Axial_DIN0207_L6.3mm_D2.5mm_P7.62mm_Horizontal"
 			(at 69.85 133.858 90)
 			(effects
@@
 			)
 		)
-		(property "Footprint" ""
+		(property "Footprint" "Resistor_THT:R_Axial_DIN0207_L6.3mm_D2.5mm_P7.62mm_Horizontal"
 			(at 69.85 47.498 90)
 			(effects
@@
 			)
 		)
-		(property "Footprint" ""
+		(property "Footprint" "Capacitor_THT:C_Disc_D3.8mm_W2.6mm_P2.50mm"
 			(at 148.59 152.4 0)
 			(effects
@@
 			)
 		)
-		(property "Footprint" ""
+		(property "Footprint" "Potentiometer_THT:Potentiometer_ACP_CA9-V10_Vertical"
 			(at 91.44 45.72 0)
 			(effects
@@
 			)
 		)
-		(property "Footprint" ""
+		(property "Footprint" "Package_DIP:DIP-14_W7.62mm_Socket"
 			(at 156.21 71.12 0)
 			(effects
@@
 			)
 		)
-		(property "Footprint" ""
+		(property "Footprint" "Resistor_THT:R_Axial_DIN0207_L6.3mm_D2.5mm_P7.62mm_Horizontal"
 			(at 64.008 140.97 90)
 			(effects
@@
 			)
 		)
-		(property "Footprint" ""
+		(property "Footprint" "Capacitor_THT:C_Disc_D3.8mm_W2.6mm_P2.50mm"
 			(at 78.74 140.97 0)
 			(effects
