File: Moog_Prodigy_Project/moog_prodigy_project/Schematics/voltage_source.kicad_sch (KiCad schematic)
At the start: 20 parts, among them J1 Conn_01x02_Socket, SW1 SW_DPST, T1 230 VAC/ 15VAC 1.5A 22W, U1 L78L12, U4 L79L12

Commit message: transformator i prekidac
Parts:
- C100, C101, C102, C103: footprint (none) -> Capacitor_THT:C_Disc_D3.8mm_W2.6mm_P2.50mm
- D102: footprint (none) -> Diode_THT:Diode_Bridge_Round_D9.0mm
- F1: footprint (none) -> Fuse:Fuse_Bourns_MF-RHT050
- F2: footprint (none) -> Fuse:Fuse_Bourns_MF-RHT100
- J1, SW1: footprint (none) -> Connector_PinSocket_2.54mm:PinSocket_1x01_P2.54mm_Horizontal
- T1: footprint (none) -> Transformer_THT:Transformer_NF_ETAL_P3324
Connections:
- net kraj_2: now reaches SW1.1, T1.2 (AB)
- net kraj_1: now reaches F1.1, SW1.3
Other:
- moved on the sheet: J1, SW1
Changed lines of the file:
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@@
+	(wire
+		(pts
+			(xy 40.64 50.8) (xy 40.64 53.34)
+		)
+		(stroke
+			(width 0)
+			(type default)
+		)
+	)
 	(wire
 		(pts
@@
 	(wire
 		(pts
+			(xy 38.1 55.88) (xy 49.53 55.88)
+		)
+		(stroke
+			(width 0)
+			(type default)
+		)
+	)
+	(wire
+		(pts
 			(xy 156.21 60.96) (xy 173.99 60.96)
 		)
@@
 	(wire
 		(pts
+			(xy 49.53 50.8) (xy 40.64 50.8)
+		)
+		(stroke
+			(width 0)
+			(type default)
+		)
+	)
+	(wire
+		(pts
 			(xy 173.99 43.18) (xy 190.5 43.18)
 		)
@@
 	(wire
 		(pts
-			(xy 60.96 55.88) (xy 72.39 55.88)
-		)
-		(stroke
-			(width 0)
-			(type default)
-		)
-	)
-	(wire
-		(pts
-			(xy 63.5 53.34) (xy 60.96 53.34)
-		)
-		(stroke
-			(width 0)
-			(type default)
-		)
-	)
-	(wire
-		(pts
-			(xy 72.39 50.8) (xy 63.5 50.8)
-		)
-		(stroke
-			(width 0)
-			(type default)
-		)
-	)
-	(wire
-		(pts
 			(xy 205.74 60.96) (xy 219.71 60.96)
 		)
@@
 	(wire
 		(pts
-			(xy 63.5 50.8) (xy 63.5 53.34)
-		)
-		(stroke
-			(width 0)
-			(type default)
-		)
-	)
-	(wire
-		(pts
 			(xy 82.55 50.8) (xy 90.17 50.8)
 		)
@@
 	(wire
 		(pts
+			(xy 40.64 53.34) (xy 38.1 53.34)
+		)
+		(stroke
+			(width 0)
+			(type default)
+		)
+	)
+	(wire
+		(pts
 			(xy 148.59 77.47) (xy 173.99 77.47)
 		)
@@
 			(width 0)
 			(type default)
+		)
+	)
+	(global_label "kraj_1"
+		(shape input)
+		(at 59.69 50.8 0)
+		(fields_autoplaced yes)
+		(effects
+			(font
+				(size 1.27 1.27)
+			)
+			(justify left)
+		)
+		(property "Intersheetrefs" "${INTERSHEET_REFS}"
+			(at 68.4204 50.8 0)
+			(effects
+				(font
+					(size 1.27 1.27)
+				)
+				(justify left)
+				(hide yes)
+			)
+		)
+	)
+	(global_label "kraj_2"
+		(shape input)
+		(at 59.69 55.88 0)
+		(fields_autoplaced yes)
+		(effects
+			(font
+				(size 1.27 1.27)
+			)
+			(justify left)
+		)
+		(property "Intersheetrefs" "${INTERSHEET_REFS}"
+			(at 68.4204 55.88 0)
+			(effects
+				(font
+					(size 1.27 1.27)
+				)
+				(justify left)
+				(hide yes)
+			)
+		)
+	)
+	(global_label "kraj_2"
+		(shape input)
+		(at 82.55 55.88 180)
+		(fields_autoplaced yes)
+		(effects
+			(font
+				(size 1.27 1.27)
+			)
+			(justify right)
+		)
+		(property "Intersheetrefs" "${INTERSHEET_REFS}"
+			(at 73.8196 55.88 0)
+			(effects
+				(font
+					(size 1.27 1.27)
+				)
+				(justify right)
+				(hide yes)
+			)
+		)
+	)
+	(global_label "kraj_1"
+		(shape input)
+		(at 82.55 50.8 180)
+		(fields_autoplaced yes)
+		(effects
+			(font
+				(size 1.27 1.27)
+			)
+			(justify right)
+		)
+		(property "Intersheetrefs" "${INTERSHEET_REFS}"
+			(at 73.8196 50.8 0)
+			(effects
+				(font
+					(size 1.27 1.27)
+				)
+				(justify right)
+				(hide yes)
+			)
 		)
 	)
@@
 			)
 		)
-		(property "Footprint" ""
+		(property "Footprint" "Transformer_THT:Transformer_NF_ETAL_P3324"
 			(at 111.76 55.88 0)
 			(effects
@@
 			)
 		)
-		(property "Footprint" ""
+		(property "Footprint" "Diode_THT:Diode_Bridge_Round_D9.0mm"
 			(at 156.21 53.34 0)
 			(effects
@@
 			)
 		)
-		(property "Footprint" ""
+		(property "Footprint" "Capacitor_THT:C_Disc_D3.8mm_W2.6mm_P2.50mm"
 			(at 190.5 52.07 0)
 			(effects
@@
 	(symbol
 		(lib_id "Switch:SW_DPST")
-		(at 77.47 53.34 0)
+		(at 54.61 53.34 0)
 		(mirror y)
 		(unit 1)
@@
 		(dnp no)
 		(property "Reference" "SW1"
-			(at 77.47 44.577 0)
+			(at 54.61 44.577 0)
 			(effects
 				(font
@@
 		)
 		(property "Value" "SW_DPST"
-			(at 77.47 47.117 0)
-			(effects
-				(font
-					(size 1.27 1.27)
-				)
-			)
-		)
-		(property "Footprint" ""
-			(at 77.47 53.34 0)
+			(at 54.61 47.117 0)
+			(effects
+				(font
+					(size 1.27 1.27)
+				)
+			)
+		)
+		(property "Footprint" "Connector_PinSocket_2.54mm:PinSocket_1x01_P2.54mm_Horizontal"
+			(at 54.61 53.34 0)
 			(effects
 				(font
@@
 		)
 		(property "Datasheet" "~"
-			(at 77.47 53.34 0)
+			(at 54.61 53.34 0)
 			(effects
 				(font
@@
 		)
 		(property "Description" ""
-			(at 77.47 53.34 0)
+			(at 54.61 53.34 0)
 			(effects
 				(font
@@
 			)
 		)
-		(property "Footprint" ""
+		(property "Footprint" "Capacitor_THT:C_Disc_D3.8mm_W2.6mm_P2.50mm"
 			(at 190.5 69.85 0)
 			(effects
@@
 			)
 		)
-		(property "Footprint" ""
+		(property "Footprint" "Fuse:Fuse_Bourns_MF-RHT050"
 			(at 93.98 52.578 90)
 			(effects
@@
 			)
 		)
-		(property "Footprint" ""
+		(property "Footprint" "Capacitor_THT:C_Disc_D3.8mm_W2.6mm_P2.50mm"
 			(at 219.71 68.58 0)
 			(effects
@@
 			)
 		)
-		(property "Footprint" ""
+		(property "Footprint" "Capacitor_THT:C_Disc_D3.8mm_W2.6mm_P2.50mm"
 			(at 219.71 52.07 0)
 			(effects
@@
 	(symbol
 		(lib_id "Connector:Conn_01x02_Socket")
-		(at 55.88 55.88 180)
+		(at 33.02 55.88 180)
 		(unit 1)
 		(exclude_from_sim no)
@@
 		(fields_autoplaced yes)
 		(property "Reference" "J1"
-			(at 56.515 47.3456 0)
+			(at 33.655 47.3456 0)
 			(effects
 				(font
@@
 		)
 		(property "Value" "Conn_01x02_Socket"
-			(at 56.515 49.8856 0)
-			(effects
-				(font
-					(size 1.27 1.27)
-				)
-			)
-		)
-		(property "Footprint" ""
-			(at 55.88 55.88 0)
+			(at 33.655 49.8856 0)
+			(effects
+				(font
+					(size 1.27 1.27)
+				)
+			)
+		)
+		(property "Footprint" "Connector_PinSocket_2.54mm:PinSocket_1x01_P2.54mm_Horizontal"
+			(at 33.02 55.88 0)
 			(effects
 				(font
@@
 		)
 		(property "Datasheet" "~"
-			(at 55.88 55.88 0)
+			(at 33.02 55.88 0)
 			(effects
 				(font
@@
 		)
 		(property "Description" ""
-			(at 55.88 55.88 0)
+			(at 33.02 55.88 0)
 			(effects
 				(font
@@
 			)
 		)
-		(property "Footprint" ""
+		(property "Footprint" "Fuse:Fuse_Bourns_MF-RHT100"
 			(at 133.35 52.578 90)
 			(effects
