File: Moog_Prodigy_Project/moog_prodigy_project/Schematics/Left_side.kicad_sch (KiCad schematic)
At the start: 58 parts, among them Q1 BC549, Q3 BC549, SW1 Switch_4x4, SW2 Switch_4x4, U2 NE5532, U2A1 OPA134, U2B1 OPA134, U3 NE5532, U4 NE5532, U5 LT1011CN8

Commit message: 27.06.2026 - dodavanje izmena sa konsultacija
Parts:
- added C37, C38, C39, C40, C41, C42, C43, C44, C45, C46, C47, C48: 100n, Capacitor_THT:CP_Radial_D5.0mm_P2.50mm, symbol Device:C
Connections:
- net +12V: now also C37.2, C39.2, C41.2, C43.2, C44.2, C48.2
- net -12V: now also C38.1, C40.2, C42.2, C45.2, C46.2, C47.2
- net Flag_ka_U6A: now also Q2.2; no longer Q2.
- net GND: now also C37.1, C38.2, C39.1, C40.1, C41.1, C42.1, C43.1, C44.1, C45.1, C46.1, C47.1, C48.1
- net at C7.1, RV4.1: now also Q2.1; no longer Q2.
- net at C7.2, R19.1, R21.2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: now also Q2.3; no longer Q2.
Other:
- note added: "1_UIA"
- note added: "2_UIB"
- note added: "32' 16' 8'"
- note added: "3_UIC"
- note added: "4_UID"
- note added: "5_UI5"
- note added: "NAPOMENA Kondenzatori: C37,C38,C39,C49,C41,C42, C43,C44,C45,C46,C47,C48 su vrednosti 100n i oni su kvalitetniji"
- note removed: "Promena oktava po položaju preklopnika: 32' krajnji levi položaj 16' srednji položaj 8' krajnji desni položaj"
- moved on the sheet: C1, C4, C7, R13, R3, R4, RV2
