File: Moog_Prodigy_Project/moog_prodigy_project/moog_prodigy_project.kicad_pcb (KiCad board)
At the start: 2 copper layers, 288.5 x 178.5 mm, 292 parts, among them J1 P2-3, J2 P2-4, J3 P2-2, J4 P2-1, J5 P2-1, J6 NJ2FD-V, J7 Conn_01x02_Socket, Q1 BC549, Q10 CA3046, Q11 BC327, Q12 BC327, Q13 BC327, Q14 BC550C, Q15 BC550C, Q16 BC550C, Q17 BC550C, Q18 BC550C, Q19 BC550C, Q3 BC549, Q4 BC107, Q7 BC549, Q8 BC556, Q9 CA3046, SW1 Switch_4x4, SW10 FINAL DECAY SWITCH, SW11 FILTER MODE, SW12 SW_DPST, SW2 Switch_4x4, SW3 Switch_4x4, SW4 SW_Slide_DPDT_3x3, SW5 Switch_4x4, SW6 Switch_1x3, SW7 Switch_4x4, SW8 SW_Slide_DPDT_3x3, SW9 FINAL DECAY SWITCH, T1 230 VAC/ 15VAC 1.5A 22W, U11 OPA234, U15 LT1469, U16 LT1228, U18 OPA184, U19 OPA184, U2 NE5532, U20 NE556N, U21 MC14007UBCP, U22 MC14007UBCP, U23 MC14007UBCP, U24 L78L12, U25 L79L12, U2A1 OPA134, U2B1 OPA134, U2B2 OPA134, U3 NE5532, U4 NE5532, U4B1 OPA134, U5 LT1011CN8, U6 NE5532, U7 NE5532, U8 LT1011CN8, U9 NE5532

Commit message: Routhed PCB final 17.05.2026
Parts:
- removed SW12: SW_DPST, 471016264143_dupli_prekidac:471016264143_2_00-3_00_
- added Double_Switch1: 200MDP1T1B1M2QEH, 200MDP1T1B1M2QEH:SW_200MDP1T1B1M2QEH, F.Cu at (73.7, -101.6)
- added U10: NE5532, NE5532AP:DIP794W45P254L1016H508Q8, F.Cu at (-234.9, -95.2)
- added U12: OPA134, OPA134PA:DIP794W45P254L959H508Q8, F.Cu at (-254.0, -133.3)
- added U13: NE5532, NE5532AP:DIP794W45P254L1016H508Q8, F.Cu at (-234.9, -114.3)
- added U14: OPA134, OPA134PA:DIP794W45P254L959H508Q8, F.Cu at (-234.9, -133.3)
- added U17: NE5532, Package_DIP:DIP-8_W7.62mm, F.Cu at (-240.0, -144.8)
- Q2, Q5, Q6: footprint BF256C:TO92127P478H483-3 -> Package_TO_SOT_THT:TO-92_Inline
- moved R110 538.7 mm to (-221.2, -113.8), turned to 90 degrees
- moved Q11 526.8 mm to (-216.2, -99.5), turned to 180 degrees
- moved R109 511.4 mm to (-206.0, -89.8), turned to 180 degrees
- moved R132 461.6 mm to (-62.5, -293.5)
- moved RV21 457.3 mm to (-41.2, -288.5)
- moved R12 453.6 mm to (-227.4, -287.2), turned to 180 degrees
- moved R127_1 451.0 mm to (-76.8, -293.5)
- moved R7 434.7 mm to (-261.0, -278.9), turned to 90 degrees
- moved R130 434.2 mm to (-120.1, -192.8)
- moved R6 434.1 mm to (-261.6, -272.2)
- moved R106 428.6 mm to (-79.5, -84.0), turned to 0 degrees
- moved U8 413.7 mm to (-177.9, -247.3), turned to -90 degrees
- moved C13 412.0 mm to (-97.5, -272.0), turned to 90 degrees
- moved R60 411.9 mm to (-195.1, -275.0)
- moved R98 410.2 mm to (-41.6, -194.8), turned to 0 degrees
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Connections:
- R7 pad 2: Net-(SW1-E) -> +12V
- SW1 pad 5: Net-(SW1-E) -> +12V
Routing:
- net +12V: track 0.00 -> 2212.7 mm, vias 0 -> 3
- net node_2: track 0.00 -> 705.5 mm, vias 0 -> 8
- net -12V: track 0.00 -> 604.3 mm, vias 0 -> 19
- net GND: track 0.00 -> 586.4 mm, vias 0 -> 22
- net Net-(C27-Pad2): track 0.00 -> 327.0 mm, vias 0 -> 1
- net Net-(U16--): track 0.00 -> 295.8 mm, vias 0 -> 6
- net THRESHOLD_2: track 0.00 -> 281.2 mm, vias 0 -> 1
- net Net-(Q15-B): track 0.00 -> 268.8 mm, vias 0 -> 5
- net Net-(R113-Pad2): track 0.00 -> 268.6 mm
- net VCA_ATTACK_PIN_12: track 0.00 -> 264.1 mm, vias 0 -> 3
- net Net-(Q10-Pad13): track 0.00 -> 260.0 mm, vias 0 -> 4
- net node_1: track 0.00 -> 251.0 mm, vias 0 -> 2
- net Net-(Q3-E): track 0.00 -> 250.7 mm, vias 0 -> 2
- net Net-(CR1-K): track 0.00 -> 239.3 mm, vias 0 -> 6
- net Net-(U6A-+): track 0.00 -> 234.8 mm, vias 0 -> 5
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- added copper zone on F.Cu, net +12V
- added copper zone on F.Cu, net -12V
- added copper zone on B.Cu, net GND
Other:
- board outline removed

Commit message: Mounting holes implementation
Parts:
- added REF**: MountingHole_3.2mm_M3, MountingHole:MountingHole_3.2mm_M3, F.Cu at (-258.4, -297.1)
- added REF**: MountingHole_3.2mm_M3, MountingHole:MountingHole_3.2mm_M3, F.Cu at (164.7, -85.2)
- added REF**: MountingHole_3.2mm_M3, MountingHole:MountingHole_3.2mm_M3, F.Cu at (-258.4, -85.1)
- added REF**: MountingHole_3.2mm_M3, MountingHole:MountingHole_3.2mm_M3, F.Cu at (164.7, -296.7)
Connections:
- R7 pad 2: +12V -> Net-(SW1-E)
- SW1 pad 5: +12V -> Net-(SW1-E)
Routing:
- net GND: track 586.4 -> 972.6 mm, vias 22 -> 35
- net -12V: track 604.3 -> 783.1 mm, vias 19 -> 28
- net Net-(SW1-E): track 44.8 -> 108.5 mm, vias 0 -> 2
- net +12V: track 2212.7 -> 2194.7 mm
