File: Moog_Prodigy_Project/moog_prodigy_project/moog_prodigy_project.kicad_pcb (KiCad board)
At the start: 2 copper layers, 387 parts, among them IC1 2N3055, IC2 2N3055, IC5 MC14007UBCP, J1 P2-3, J2 P2-4, J3 P2-2, J4 P2-1, J5 P2-1, J6 NJ2FD-V, Q11 BC549, Q12 BC327, Q13 BC327, Q14 BC550C, Q15 BC550C, Q16 BC550C, Q17 BC550C, Q18 BC550C, Q19 BC550C, Q2 E112, Q20 BC549, Q21 BC549, Q4 BC549, Q5 E112, Q6 E112, Q7 BC549, Q8 BC549, SW1 Switch_4x4, SW11 FILTER MODE, SW12 FINAL DECAY SWITCH, SW13 FINAL DECAY SWITCH, SW1_0 200MDP1T1B1M2QEH, SW2 Switch_4x4, SW3 Switch_4x4, SW4 SW_Slide_DPDT_3x3, SW5 Switch_4x4, SW6 Switch_1x3, SW7 Switch_4x4, SW8 SW_Slide_DPDT_3x3, T2 230VAC / 2x15VAC 0A53 16VA, U1 NE5532, U11 OPA234, U12 OPA134, U13 NE5532, U14 OPA134, U15 LT1469, U16 LT1228, U17 NE5532, U18 OPA184, U19 OPA184, U2 NE5532, U20 NE556N, U21 MC14007UBCP, U22 MC14007UBCP, U23 MC14007UBCP, U24 LM7812, U25 LM7912, U26 OPA184, U27 OPA184, U2A1 OPA134, U2B1 OPA134, U2B2 OPA134, U3 NE5532, U4 NE5532, U4B1 OPA134, U5 LT1011CN8, U6 NE5532, U7 NE5532, U8 LT1011CN8, U9 NE5532

Commit message: uklonjeni pojedini potenciometri, radjeno merenje ploce
Parts:
- removed C90: 10u, Capacitor_THT:CP_Radial_D5.0mm_P2.50mm
- removed RV18: 1M, Potentiometer_THT:Potentiometer_ACP_CA9-V10_Vertical
- moved J6 63.8 mm to (3.05, -159.5), turned to 0 degrees
Routing:
- net node_8: track 204.1 -> 167.7 mm, vias 14 -> 11
- net node_9: track 59.9 -> 47.3 mm

Commit message: Update tracks 16.07.2026
Routing:
- net THRESHOLD_2: track 285.8 -> 606.1 mm, vias 16 -> 2
- net Net-(R85-Pad1): track 431.7 -> 178.9 mm
- net Net-(U11A--): track 153.2 -> 346.8 mm, vias 4 -> 9
- net Net-(SW13-B): track 329.0 -> 162.5 mm, vias 0 -> 3
- net node_8: track 167.7 -> 16.8 mm, vias 11 -> 0
- net Net-(R141-Pad1): track 318.4 -> 433.1 mm, vias 17 -> 3
- net Net-(R71-Pad1): track 172.9 -> 279.4 mm, vias 0 -> 7
- net -12V: track 1129.6 -> 1230.9 mm, vias 30 -> 4
- net Net-(J6-PadS): track 85.1 -> 164.2 mm, vias 1 -> 2
- net Flag to R87: track 147.3 -> 225.6 mm, vias 0 -> 7
- net Net-(R142-Pad2): track 428.0 -> 506.1 mm, vias 6 -> 10
- net Net-(U16--): track 122.3 -> 198.7 mm
- net Net-(SW6-C): track 162.2 -> 236.9 mm, vias 15 -> 11
- net Net-(R35-Pad2): track 76.6 -> 150.0 mm, vias 5 -> 11
- net Net-(D8-A): track 104.3 -> 176.1 mm, vias 2 -> 11
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- added copper zone on B.Cu, net +12V
- added copper zone on F.Cu, net +12V
- added copper zone on B.Cu, net GND
