File: Moog_Prodigy_Project/moog_prodigy_project/Left_side_pt2.kicad_sch (KiCad schematic)
At the start: 64 parts, among them J7 Conn_01x02_Socket, Q4 BC107, Q7 BC549, SW3 Switch_4x4, SW4 SW_Slide_DPDT_3x3, SW5 Switch_4x4, U2B2 OPA134, U4B1 OPA134, U6 NE5532, U7 NE5532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

Commit message: 27.06.2026 - dodavanje izmena sa konsultacija
Parts:
- added C49, C50, C51, C52, C53, C54, C55, C56, C57, C58: 100n, Capacitor_THT:CP_Radial_D5.0mm_P2.50mm, symbol Device:C
Connections:
- net +12V: now also C49.2, C51.2, C53.2, C55.2, C57.2
- net -12V: now also C50.2, C52.2, C54.2, C56.2, C58.2
- net GND: now also C49.1, C50.1, C51.1, C52.1, C53.1, C54.1, C55.1, C56.1, C57.1, C58.1
- net at C18.1, R54.1, R55.1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: now also Q6.1; no longer Q6.
- net at C17.1, Q5., R52.1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: now also Q6.2; no longer Q6.
- net at C17.2, Q5., R54.2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: now also Q6.3; no longer Q6.
Other:
- note added: "16' 8' 4'"
- note added: "1_UIA"
- note added: "2_UIB"
- note added: "3_UIC"
- note added: "4_UID"
- note added: "5_UIE"
- note added: "NAPOMENA Kondenzatori: C49,C50,C51,C52,C53, C54,C55,C56,C57,C58 su vrednosti 100n i oni su kvalitetniji"
- note removed: "Promena oktava po položaju preklopnika: 16' - krajnji levi položaj 8' - srednji položaj 4' - krajnji desni položaj"
- moved on the sheet: C11, C12, R38, R39, RV7
