File: Moog_Prodigy_Project/moog_prodigy_project/ledder_transistors.kicad_sch (KiCad schematic)
At the start: 26 parts, among them Q104 BC550C, Q105 BC550C, Q106 BC550C, Q107 BC550C, Q108 BC550C, Q109 BC550C, SW100 FILTER MODE

Commit message: PCB priprema i fix gresaka
Parts:
- RV105, RV107: footprint Resistor_THT:R_Axial_DIN0207_L6.3mm_D2.5mm_P7.62mm_Horizontal -> Potentiometer_THT:Potentiometer_Bourns_3339P_Vertical_HandSoldering
Changed lines of the file:
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@@
 			)
 		)
-		(property "Footprint" "Resistor_THT:R_Axial_DIN0207_L6.3mm_D2.5mm_P7.62mm_Horizontal"
+		(property "Footprint" "Potentiometer_THT:Potentiometer_Bourns_3339P_Vertical_HandSoldering"
 			(at 120.65 67.31 0)
 			(effects
@@
 			)
 		)
-		(property "Footprint" "Resistor_THT:R_Axial_DIN0207_L6.3mm_D2.5mm_P7.62mm_Horizontal"
+		(property "Footprint" "Potentiometer_THT:Potentiometer_Bourns_3339P_Vertical_HandSoldering"
 			(at 157.48 118.11 0)
 			(effects

Commit message: problemi sa ca3096, multiplicirani footprintovi
Parts:
- RV21: renamed from RV107; footprint Potentiometer_THT:Potentiometer_Bourns_3339P_Vertical_HandSoldering -> Potentiometer_THT:Potentiometer_ACP_CA9-V10_Vertical
- renumbered C108 to C29, C109 to C30, CP103 to CP6, Q104 to Q14, Q106 to Q15, Q108 to Q16, Q105 to Q17, Q107 to Q18, Q109 to Q19, R108_2 to R108_1, R125_2 to R125_1, R126_2 to R126_1, R108 to R127, R127_2 to R127_1, R125 to R128, R128_2 to R128_1, R126 to R129, R127 to R130, R128 to R131, R130 to R132, R129 to R133, RV106 to RV22, RV108 to RV23, RV105 to RV24, SW100 to SW11

Commit message: Fix 1 nakon review-a 27.05.2026
Connections:
- net node_4: now also Q16. (E); no longer Q16.3 (E)
- net node_5: now also Q19. (E); no longer Q19.3 (E)
- net node_6: now also Q14. (E); no longer Q14.1 (C)
- net node_7: now also Q17. (E); no longer Q17.1 (C)
- net at R128.2, R129.1: now also Q14. (E), Q17. (E); no longer Q14.2 (B), Q17.2 (B)
- net at R129.2, R130.1: now also Q15. (E), Q18. (E); no longer Q15.2 (B), Q18.2 (B)
- net at R130.2, R131.1: now also Q16. (E), Q19. (E); no longer Q16.2 (B), Q19.2 (B)
- new net: C29.2, Q17. (E), Q18. (E)
- new net: C29.1, Q14. (E), Q15. (E)
- new net: C30.1, Q15. (E), Q16. (E)
- new net: C30.2, Q18. (E), Q19. (E)
Changed lines of the file:
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@@
 	(generator_version "9.0")
 	(paper "A4")
+	(title_block
+		(rev "Marjan Urekar")
+		(comment 1 "Fakultet tehničkih nauka")
+		(comment 2 "Univerzitet u Novom Sadu")
+		(comment 3 "Merno-Informacioni sistemi")
+	)
 	(text "FILTER\nCUTOFF FREQ"
 		(exclude_from_sim no)
@@
 	)
 	(symbol
+		(lib_name "BC550_2")
 		(lib_id "Transistor_BJT:BC550")
 		(at 82.55 66.04 0)
@@
 			)
 		)
-		(pin "1"
+		(pin ""
 		)
-		(pin "3"
+		(pin ""
 		)
-		(pin "2"
+		(pin ""
 		)
 		(instances
@@
 	)
 	(symbol
+		(lib_name "BC550_4")
 		(lib_id "Transistor_BJT:BC550")
 		(at 64.77 86.36 0)
@@
 			)
 		)
-		(pin "1"
+		(pin ""
 		)
-		(pin "3"
+		(pin ""
 		)
-		(pin "2"
+		(pin ""
 		)
 		(instances
@@
 	)
 	(symbol
+		(lib_name "BC550_1")
 		(lib_id "Transistor_BJT:BC550")
 		(at 64.77 66.04 0)
@@
 			)
 		)
-		(pin "1"
+		(pin ""
 		)
-		(pin "3"
+		(pin ""
 		)
-		(pin "2"
+		(pin ""
 		)
 		(instances
@@
 	)
 	(symbol
+		(lib_name "BC550_3")
 		(lib_id "Transistor_BJT:BC550")
 		(at 82.55 86.36 0)
@@
 			)
 		)
-		(pin "1"
+		(pin ""
 		)
-		(pin "3"
+		(pin ""
 		)
-		(pin "2"
+		(pin ""
 		)
 		(instances
@@
 			)
 		)
-		(pin "1"
+		(pin ""
 		)
-		(pin "3"
+		(pin ""
 		)
-		(pin "2"
+		(pin ""
 		)
 		(instances
@@
 	)
 	(symbol
+		(lib_name "BC550_5")
 		(lib_id "Transistor_BJT:BC550")
 		(at 64.77 105.41 0)
@@
 			)
 		)
-		(pin "1"
+		(pin ""
 		)
-		(pin "3"
+		(pin ""
 		)
-		(pin "2"
+		(pin ""
 		)
 		(instances

Commit message: Latest checkpoints update 05.06.2026
Connections:
- net GND: now also CP6.; no longer CP6.2
- net node_1: now also CP6.; no longer CP6.1
- new net: C29.2, Q17. (E), Q18. (E)
- new net: C29.1, Q14. (E), Q15. (E)
Other:
- moved on the sheet: C29, C30, Q14, Q15, Q16, Q17, Q18, Q19, R108_1, R125_1, R126_1, R127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

Commit message: 27.06.2026 - dodavanje izmena sa konsultacija
Connections:
- new net: C29.2, Q17. (E), Q18. (E)
- new net: C29.1, Q14. (E), Q15. (E)
Changed lines of the file:
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@@
 		(comment 1 "Fakultet tehničkih nauka")
 		(comment 2 "Univerzitet u Novom Sadu")
-		(comment 3 "Merno-Informacioni sistemi")
+		(comment 3 "Merno-Informacioni sistemi ")
 	)
 	(text "FILTER\nCUTOFF FREQ"
