File: Moog_Prodigy_Project/moog_prodigy_project/ledder_transistors.kicad_sch (KiCad schematic)
At the start: 26 parts, among them Q14 BC550C, Q15 BC550C, Q16 BC550C, Q17 BC550C, Q18 BC550C, Q19 BC550C, SW11 FILTER MODE

Commit message: Dodao u napomenu za linearne i logaritamske potenciometre, NE555 i sa 4007 semom spojena u jedno, dodati kvalitetni kondenzatori, ostao simbol za 4007 da izenim kao sto je jocke
Connections:
- new net: C29.2, Q17. (E), Q18. (E)
- new net: C29.1, Q14. (E), Q15. (E)
Other:
- note added: "FILTER SCALE TRIM"
- note added: "NAPOMENA Ponteciometri: Linearni:RV22,RV23"
- title: (none) -> Ledder
Changed lines of the file:
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@@
 	(paper "A4")
 	(title_block
+		(title "Ledder")
+		(date "27.05.2026")
 		(rev "Marjan Urekar")
 		(comment 1 "Fakultet tehničkih nauka")
 		(comment 2 "Univerzitet u Novom Sadu")
 		(comment 3 "Merno-Informacioni sistemi ")
+		(comment 4 "Miodrag Babić E1 87/2023")
+	)
+	(text "NAPOMENA\nPonteciometri:\nLinearni:RV22,RV23"
+		(exclude_from_sim no)
+		(at 181.356 158.242 0)
+		(effects
+			(font
+				(size 1.27 1.27)
+			)
+			(justify left)
+		)
 	)
 	(text "FILTER\nCUTOFF FREQ"
@@
 		(effects
 			(font
+				(size 1.27 1.27)
+			)
+			(justify bottom)
+		)
+	)
+	(text "FILTER SCALE\nTRIM"
+		(exclude_from_sim no)
+		(at 140.462 85.09 0)
+		(effects
+			(font

Commit message: MOOG prodigy final 03.07.2026
Connections:
- new net: C29.2, Q17. (E), Q18. (E)
- new net: C29.1, Q14. (E), Q15. (E)
Other:
- note added: "NAPOMENA 1 Otpornici cija je vrednost: 63K4, 18K2, 4K75, 6K81, 51M, 2.4M su otpornici iz E96 serije (1%) Ostali orpotnici su iz serije E24 (5%)"
- note added: "NAPOMENA 2 Ponteciometri: Linearni:RV22,RV23"
- note removed: "NAPOMENA Ponteciometri: Linearni:RV22,RV23"
Changed lines of the file:
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@@
 		(comment 4 "Miodrag Babić E1 87/2023")
 	)
-	(text "NAPOMENA\nPonteciometri:\nLinearni:RV22,RV23"
+	(text "NAPOMENA 2\nPonteciometri:\nLinearni:RV22,RV23"
 		(exclude_from_sim no)
-		(at 181.356 158.242 0)
+		(at 215.9 157.988 0)
 		(effects
 			(font
 				(size 1.27 1.27)
+				(thickness 0.254)
+				(bold yes)
 			)
 			(justify left)
@@
 		)
 	)
+	(text "NAPOMENA 1\nOtpornici cija je vrednost:\n63K4, 18K2, 4K75, 6K81, 51M, 2.4M\nsu otpornici iz E96 serije (1%)\nOstali orpotnici su iz serije E24 (5%)"
+		(exclude_from_sim no)
+		(at 176.784 159.766 0)
+		(effects
+			(font
+				(size 1.27 1.27)
+				(thickness 0.254)
+				(bold yes)
+			)
+			(justify left)
+		)
+	)

Commit message: Moog prodigy fix 3
Parts:
- removed C29, C30: 27n, Capacitor_THT:C_Disc_D3.8mm_W2.6mm_P2.50mm, symbol Device:C_Small
- removed CP6: 220u, Capacitor_THT:CP_Radial_D5.0mm_P2.50mm, symbol elektrolitski:elektrolit
- removed Q14, Q15, Q16, Q17, Q18, Q19: BC550C, Package_TO_SOT_THT:TO-92_Inline, symbol Transistor_BJT:BC550
- removed R108_1: 200, Resistor_THT:R_Axial_DIN0207_L6.3mm_D2.5mm_P7.62mm_Horizontal, symbol Device:R
- removed R125_1: 953, Resistor_THT:R_Axial_DIN0207_L6.3mm_D2.5mm_P7.62mm_Horizontal, symbol Device:R
- removed R126_1: 51K, Resistor_THT:R_Axial_DIN0207_L6.3mm_D2.5mm_P7.62mm_Horizontal, symbol Device:R
- removed R127, R128, R129, R130, R131: 150, Resistor_THT:R_Axial_DIN0207_L6.3mm_D2.5mm_P7.62mm_Horizontal, symbol Device:R
- removed R127_1: 60K4, Resistor_THT:R_Axial_DIN0207_L6.3mm_D2.5mm_P7.62mm_Horizontal, symbol Device:R
- removed R128_1: 36K, Resistor_THT:R_Axial_DIN0207_L6.3mm_D2.5mm_P7.62mm_Horizontal, symbol Device:R
- removed R132, R133: 100K, Resistor_THT:R_Axial_DIN0207_L6.3mm_D2.5mm_P7.62mm_Horizontal, symbol Device:R
- removed RV21: 100K, Potentiometer_THT:Potentiometer_ACP_CA9-V10_Vertical, symbol Device:R_Potentiometer_Trim
- removed RV22, RV23: 50K, Potentiometer_THT:Potentiometer_ACP_CA9-V10_Vertical, symbol Device:R_Potentiometer
- removed RV24: 250, Potentiometer_THT:Potentiometer_Bourns_3339P_Vertical_HandSoldering, symbol Device:R_Potentiometer_Trim
- removed SW11: FILTER MODE, ATE1D-2M3-10-Z_1x2:SW_ATE1D-2M3-10-Z, symbol Switch:SW_SPDT
Connections:
- no-connect marks 1 -> 0
Other:
- note removed: "CONTOUR AMOUNT"
- note removed: "FILTER CUTOFF FREQ"
- note removed: "FILTER SCALE TRIM"
- note removed: "FREQ TRIM"
- note removed: "NAPOMENA 1 Otpornici cija je vrednost: 63K4, 18K2, 4K75, 6K81, 51M, 2.4M su otpornici iz E96 serije (1%) Ostali orpotnici su iz serije E24 (5%)"
- note removed: "NAPOMENA 2 Ponteciometri: Linearni:RV22,RV23"
- note removed: "OFF"
- note removed: "ON"
