File: Moog_Prodigy_Project/moog_prodigy_project/moog_prodigy_project.kicad_sch (KiCad schematic)
At the start: 0 parts

Commit message: Spajanje projekta final 1
Other:
- removed sheet Right_side
- added sheet 3046 (ledder.kicad_sch)
- added sheet 4007 (4007_mosfets.kicad_sch)
- added sheet Left_side_pt2 (Left_side_pt2.kicad_sch)
- added sheet Left_side_pt3 (Left_side_pt3.kicad_sch)
- added sheet dual_timer (dual_timer.kicad_sch)
- added sheet ledder (ledder_transistors.kicad_sch)
- added sheet vca_attack (vca_attack.kicad_sch)
- added sheet voltage_source (voltage_source.kicad_sch)
