File: Moog_Prodigy_Project/moog_prodigy_project/moog_prodigy_project.kicad_sch (KiCad schematic)
At the start: 0 parts

Commit message: Dodao u napomenu za linearne i logaritamske potenciometre, NE555 i sa 4007 semom spojena u jedno, dodati kvalitetni kondenzatori, ostao simbol za 4007 da izenim kao sto je jocke
Other:
- removed sheet dual_timer
- removed sheet vca_attack
Changed lines of the file:
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@@
-	)
-	(sheet
-		(at 96.52 64.77)
-		(size 59.69 25.4)
-		(exclude_from_sim no)
-		(in_bom yes)
-		(on_board yes)
-		(dnp no)
-		(fields_autoplaced yes)
-		(stroke
-			(width 0.1524)
-			(type solid)
-		)
-		(fill
-			(color 0 0 0 0.0000)
-		)
-		(property "Sheetname" "dual_timer"
-			(at 96.52 64.0584 0)
-			(effects
-				(font
-					(size 1.27 1.27)
-				)
-				(justify left bottom)
-			)
-		)
-		(property "Sheetfile" "dual_timer.kicad_sch"
-			(at 96.52 90.7546 0)
-			(effects
-				(font
-					(size 1.27 1.27)
-				)
-				(justify left top)
-			)
-		)
-		(instances
-			(project "moog_prodigy_project"
-				(path "/db469bdb-b6c3-4a16-9199-d4e6b8d556e8"
-					(page "7")
-				)
-			)
-		)
 	)
 	(sheet
@@
 				)
 			)
-		)
-	)
-	(sheet
-		(at 96.52 102.87)
-		(size 59.69 25.4)
-		(exclude_from_sim no)
-		(in_bom yes)
-		(on_board yes)
-		(dnp no)
-		(fields_autoplaced yes)
-		(stroke
-			(width 0.1524)
-			(type solid)
-		)
-		(fill
-			(color 0 0 0 0.0000)
-		)
-		(property "Sheetname" "vca_attack"
-			(at 96.52 102.1584 0)
-			(effects
-				(font
-					(size 1.27 1.27)
-				)
-				(justify left bottom)
-			)
-		)
-		(property "Sheetfile" "vca_attack.kicad_sch"
-			(at 96.52 128.8546 0)
-			(effects
-				(font
-					(size 1.27 1.27)
-				)
-				(justify left top)
-			)
-		)
-		(instances
-			(project "moog_prodigy_project"
-				(path "/db469bdb-b6c3-4a16-9199-d4e6b8d556e8"
-					(page "9")
-				)
-			)

Commit message: Moog prodigy fix 3
Other:
- removed sheet ledder
Changed lines of the file:
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@@
-	)
-	(sheet
-		(at 163.195 64.77)
-		(size 59.055 25.4)
-		(exclude_from_sim no)
-		(in_bom yes)
-		(on_board yes)
-		(dnp no)
-		(fields_autoplaced yes)
-		(stroke
-			(width 0.1524)
-			(type solid)
-		)
-		(fill
-			(color 0 0 0 0.0000)
-		)
-		(property "Sheetname" "ledder"
-			(at 163.195 64.0584 0)
-			(effects
-				(font
-					(size 1.27 1.27)
-				)
-				(justify left bottom)
-			)
-		)
-		(property "Sheetfile" "ledder_transistors.kicad_sch"
-			(at 163.195 90.7546 0)
-			(effects
-				(font
-					(size 1.27 1.27)
-				)
-				(justify left top)
-			)
-		)
-		(instances
-			(project "moog_prodigy_project"
-				(path "/db469bdb-b6c3-4a16-9199-d4e6b8d556e8"
-					(page "8")
-				)
-			)
-		)
 	)
 	(sheet
