File: Moog_Prodigy_Project/moog_prodigy_project/dual_timer.kicad_sch (KiCad schematic)
At the start: 3 parts, among them U20 NE556N

Commit message: Dodao u napomenu za linearne i logaritamske potenciometre, NE555 i sa 4007 semom spojena u jedno, dodati kvalitetni kondenzatori, ostao simbol za 4007 da izenim kao sto je jocke
Parts:
- removed CP5: 10u, Capacitor_THT:CP_Radial_D5.0mm_P2.50mm, symbol elektrolitski:elektrolit
- removed R126: 100, Resistor_THT:R_Axial_DIN0207_L6.3mm_D2.5mm_P7.62mm_Horizontal, symbol Device:R
- removed U20: NE556N, NE556N:DIP794W45P254L1930H508Q14, symbol NE556N:NE556N
Connections:
- no-connect marks 4 -> 0
