File: Moog_Prodigy_Project/moog_prodigy_project/Left_side_pt3.kicad_sch (KiCad schematic)
At the start: 68 parts, among them J1 P2-3, J2 P2-4, J3 P2-2, J4 P2-1, J5 P2-1, SW6 Switch_1x3, SW7 Switch_4x4, SW8 SW_Slide_DPDT_3x3, U10 NE5532, U11 OPA234, U12 OPA134, U13 NE5532, U14 OPA134, U9 NE5532

Commit message: Dodao u napomenu za linearne i logaritamske potenciometre, NE555 i sa 4007 semom spojena u jedno, dodati kvalitetni kondenzatori, ostao simbol za 4007 da izenim kao sto je jocke
Other:
- note added: "NAPOMENA Kondenzatori: C59,C60,C61,C62,C63,C64, C65,C66,C67,C68,C69,C70 su vrednosti 100n i oni su kvalitetniji Potenciometari: Linearni: Logaritamski: RV11"
- note added: "TUNE"
- note removed: "NAPOMENA Kondenzatori: C59,C60,C61,C62,C63,C64, C65,C66,C67,C68,C69,C70 su vrednosti 100n i oni su kvalitetniji"
Changed lines of the file:
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@@
 		)
 	)
-	(text "NAPOMENA\nKondenzatori:\nC59,C60,C61,C62,C63,C64,\nC65,C66,C67,C68,C69,C70\nsu vrednosti 100n i oni su kvalitetniji"
+	(text "NAPOMENA\nKondenzatori:\nC59,C60,C61,C62,C63,C64,\nC65,C66,C67,C68,C69,C70\nsu vrednosti 100n i oni su kvalitetniji\n\nPotenciometari:\nLinearni:\nLogaritamski: RV11"
 		(exclude_from_sim no)
-		(at 177.038 158.496 0)
+		(at 193.548 155.956 0)
 		(effects
 			(font
@@
 		(effects
 			(font
+				(size 1.27 1.27)
+				(thickness 0.254)
+				(bold yes)
+			)
+		)
+	)
+	(text "TUNE"
+		(exclude_from_sim no)
+		(at 97.536 121.92 0)
+		(effects
+			(font

Commit message: Update seme final 1
Connections:
- net to_VCA/VCF: no longer 1_UI4.
- no-connect marks 11 -> 9
Other:
- moved on the sheet: 1_UI4A, 4_UI4D, C67, C70, CR1, CR2, R83, R84, R85, R86, R88, R89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

Commit message: MOOG prodigy final 03.07.2026
Parts:
- R69: value 2.5M -> 2M5
- R77: value 4.7KΩ -> 4K7 1%
- R85: value 5.1M -> 5M1
- R90: value 2.4M -> 2M4 1%
Connections:
- no-connect marks 9 -> 10
Other:
- note added: "NAPOMENA 1 Kondenzatori: C59,C60,C61,C62,C63,C64, C65,C66,C67,C68,C69,C70 su vrednosti 100n i oni su kvalitetniji Potenciometari: Linearni: Logaritamski: RV11"
- note added: "NAPOMENA 2 Otpornici cija je vrednost: 63K4, 18K2, 4K75, 6K81, 51M, 2.4M su otpornici iz E96 serije (1%) Ostali orpotnici su iz serije E24 (5%)"
- note added: "Neiskorisceni FET-ovi iz 4007: - 1_UI14A - 4_UI4D"
- note removed: "NAPOMENA Kondenzatori: C59,C60,C61,C62,C63,C64, C65,C66,C67,C68,C69,C70 su vrednosti 100n i oni su kvalitetniji Potenciometari: Linearni: Logaritamski: RV11"
- moved on the sheet: 1_UI4A, 4_UI4D
Changed lines of the file:
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@@
 		(comment 4 "Jovan Mastelica E1 105/2023")
 	)
+	(text "Neiskorisceni FET-ovi iz 4007:\n- 1_UI14A\n- 4_UI4D\n"
+		(exclude_from_sim no)
+		(at 253.492 142.494 0)
+		(effects
+			(font
+				(size 1.27 1.27)
+				(thickness 0.254)
+				(bold yes)
+			)
+			(justify left)
+		)
+	)
 	(text "Oblik signala po položaju preklopnika\n\nTrougao        Četvrtka "
 		(exclude_from_sim no)
@@
 			(font
 				(size 1.27 1.27)
+				(thickness 0.254)
+				(bold yes)
 			)
 		)
@@
 		)
 	)
-	(text "NAPOMENA\nKondenzatori:\nC59,C60,C61,C62,C63,C64,\nC65,C66,C67,C68,C69,C70\nsu vrednosti 100n i oni su kvalitetniji\n\nPotenciometari:\nLinearni:\nLogaritamski: RV11"
+	(text "NAPOMENA 1\nKondenzatori:\nC59,C60,C61,C62,C63,C64,\nC65,C66,C67,C68,C69,C70\nsu vrednosti 100n i oni su kvalitetniji\n\nPotenciometari:\nLinearni:\nLogaritamski: RV11"
 		(exclude_from_sim no)
-		(at 193.548 155.956 0)
+		(at 176.784 156.21 0)
 		(effects
 			(font
@@
 		)
 	)
+	(text "NAPOMENA 2\nOtpornici cija je vrednost:\n63K4, 18K2, 4K75, 6K81, 51M, 2.4M\nsu otpornici iz E96 serije (1%)\nOstali orpotnici su iz serije E24 (5%)"
+		(exclude_from_sim no)
+		(at 216.154 152.146 0)
+		(effects
+			(font
+				(size 1.27 1.27)
+				(thickness 0.254)
+				(bold yes)
+			)
+			(justify left)
+		)
+	)
 	(text "MOD\nAMOUNT"
 		(exclude_from_sim no)
@@
 	)
 	(no_connect
-		(at 276.86 154.94)
+		(at 276.86 163.83)
 	)
 	(no_connect
-		(at 264.16 143.51)
+		(at 265.43 154.94)
 	)
 	(no_connect
-		(at 276.86 137.16)
+		(at 276.86 146.05)
 	)
 	(no_connect
@@
 	)
 	(no_connect
-		(at 69.85 121.92)
+		(at 71.12 121.92)
 	)
 	(no_connect
-		(at 254 143.51)
+		(at 255.27 154.94)
 	)
 	(no_connect
 		(at 180.34 127)
 	)
+	(no_connect
+		(at 260.35 147.32)
+	)
 	(wire
 		(pts
@@
 	(wire
 		(pts
-			(xy 104.14 63.5) (xy 104.14 59.69)
+			(xy 104.14 58.42) (xy 104.14 63.5)
 		)
 		(stroke
@@
 			)
 		)
-		(property "Value" "5.1M"
+		(property "Value" "5M1"
 			(at 110.49 117.094 90)
 			(effects
@@
 			)
 		)
-		(property "Value" "2.4M"
+		(property "Value" "2M4 1%"
 			(at 153.67 102.108 90)
 			(effects
@@
 	(symbol
 		(lib_id "Transistor_FET:4007_Novi")
-		(at 104.14 52.07 270)
+		(at 104.14 55.88 90)
 		(unit 2)
 		(exclude_from_sim no)
@@
 		(dnp no)
 		(property "Reference" "2_UI4"
-			(at 104.14 48.26 90)
+			(at 104.14 50.038 90)
 			(effects
 				(font
@@
 		)
 		(property "Value" "4007"
-			(at 104.14 50.8 90)
+			(at 104.14 47.752 90)
 			(effects
 				(font
@@
 		)
 		(property "Footprint" "Package_DIP:DIP-14_W7.62mm_Socket"
-			(at 104.14 52.07 0)
+			(at 104.14 55.88 0)
 			(effects
 				(font
@@
 		)
 		(property "Datasheet" ""
-			(at 104.14 52.07 0)
+			(at 104.14 55.88 0)
 			(effects
 				(font
@@
 		)
 		(property "Description" ""
-			(at 104.14 52.07 0)
+			(at 104.14 55.88 0)
 			(effects
 				(font
@@
 			)
 		)
-		(property "Value" "4.7KΩ"
+		(property "Value" "4K7 1%"
 			(at 86.36 56.134 90)
 			(effects
@@
 		(lib_name "4007_Novi_1")
 		(lib_id "Transistor_FET:4007_Novi")
-		(at 259.08 143.51 90)
+		(at 260.35 154.94 90)
 		(unit 1)
 		(exclude_from_sim no)
@@
 		(fields_autoplaced yes)
 		(property "Reference" "1_UI4"
-			(at 259.08 147.32 90)
+			(at 260.35 158.75 90)
 			(effects
 				(font
@@
 		)
 		(property "Value" "4007"
-			(at 259.08 144.78 90)
+			(at 260.35 156.21 90)
 			(effects
 				(font
@@
 		)
 		(property "Footprint" "Package_DIP:DIP-14_W7.62mm_Socket"
-			(at 259.08 143.51 0)
+			(at 260.35 154.94 0)
 			(effects
 				(font
@@
 		)
 		(property "Datasheet" ""
-			(at 259.08 143.51 0)
+			(at 260.35 154.94 0)
 			(effects
 				(font
@@
 		)
 		(property "Description" ""
-			(at 259.08 143.51 0)
+			(at 260.35 154.94 0)
 			(effects
 				(font
@@
 		(lib_name "4007_Novi_4")
 		(lib_id "Transistor_FET:4007_Novi")
-		(at 86.36 118.11 180)
+		(at 82.55 116.84 0)
 		(unit 5)
 		(exclude_from_sim no)
@@
 		(dnp no)
 		(property "Reference" "5_UI4"
-			(at 89.408 118.11 0)
+			(at 81.788 121.666 0)
 			(effects
 				(font
@@
 		)
 		(property "Value" "4007"
-			(at 89.408 120.65 0)
+			(at 82.296 123.952 0)
 			(effects
 				(font
@@
 		)
 		(property "Footprint" "Package_DIP:DIP-14_W7.62mm_Socket"
-			(at 86.36 118.11 0)
+			(at 82.55 116.84 0)
 			(effects
 				(font
@@
 		)
 		(property "Datasheet" ""
-			(at 86.36 118.11 0)
+			(at 82.55 116.84 0)
 			(effects
 				(font
@@
 		)
 		(property "Description" ""
-			(at 86.36 118.11 0)
+			(at 82.55 116.84 0)
 			(effects
 				(font
@@
 		(lib_name "4007_Novi_2")
 		(lib_id "Transistor_FET:4007_Novi")
-		(at 276.86 149.86 180)
+		(at 276.86 158.75 180)
 		(unit 4)
 		(exclude_from_sim no)
@@
 		(dnp no)
 		(property "Reference" "4_UI4"
-			(at 280.67 149.352 0)
+			(at 280.67 158.242 0)
 			(effects
 				(font
@@
 		)
 		(property "Value" "4007"
-			(at 280.67 151.892 0)
+			(at 280.67 160.782 0)
 			(effects
 				(font
@@
 		)
 		(property "Footprint" "Package_DIP:DIP-14_W7.62mm_Socket"
-			(at 276.86 149.86 0)
+			(at 276.86 158.75 0)
 			(effects
 				(font
@@
 		)
 		(property "Datasheet" ""
-			(at 276.86 149.86 0)
+			(at 276.86 158.75 0)
 			(effects
 				(font
@@
 		)
 		(property "Description" ""
-			(at 276.86 149.86 0)
+			(at 276.86 158.75 0)
 			(effects
 				(font
@@
 			)
 		)
-		(property "Value" "2.5M"
+		(property "Value" "2M5"
 			(at 37.084 101.092 90)
 			(effects
@@
 	(symbol
 		(lib_id "power:GND")
-		(at 69.85 132.08 0)
+		(at 71.12 132.08 0)
 		(unit 1)
 		(exclude_from_sim no)
@@
 		(dnp no)
 		(property "Reference" "#PWR091"
-			(at 69.85 138.43 0)
+			(at 71.12 138.43 0)
 			(effects
 				(font
@@
 		)
 		(property "Value" "GND"
-			(at 69.85 135.636 0)
+			(at 71.12 135.636 0)
 			(effects
 				(font
@@
 		)
 		(property "Footprint" ""
-			(at 69.85 132.08 0)
+			(at 71.12 132.08 0)
 			(effects
 				(font
@@
 		)
 		(property "Datasheet" ""
-			(at 69.85 132.08 0)
+			(at 71.12 132.08 0)
 			(effects
 				(font
@@
 		)
 		(property "Description" "Power symbol creates a global label with name \"GND\" , ground"
-			(at 69.85 132.08 0)
+			(at 71.12 132.08 0)
 			(effects
 				(font
