File: Moog_Prodigy_Project/moog_prodigy_project/voltage_source.kicad_sch (KiCad schematic)
At the start: 24 parts, among them T2 230 VAC/ 15VAC 1.5A 22W, U24 LM78L12, U25 LM79L12

Commit message: Moog prodigy fix 3
Parts:
- T2: value 230 VAC/ 15VAC 1.5A 22W -> 230 VAC/ 15VAC 1A5 22W
Changed lines of the file:
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@@
+	)
+	(symbol
+		(lib_name "LED_1")
+		(lib_id "Device:LED")
+		(at 245.11 74.93 90)
+		(unit 1)
+		(exclude_from_sim no)
+		(in_bom yes)
+		(on_board yes)
+		(dnp no)
+		(property "Reference" "D7"
+			(at 249.682 75.438 90)
+			(effects
+				(font
+					(size 1.27 1.27)
+				)
+				(justify left)
+			)
+		)
+		(property "Value" "RED LED"
+			(at 253.492 80.772 90)
+			(effects
+				(font
+					(size 1.27 1.27)
+				)
+				(justify left)
+			)
+		)
+		(property "Footprint" ""
+			(at 245.11 74.93 0)
+			(effects
+				(font
+					(size 1.27 1.27)
+				)
+				(hide yes)
+			)
+		)
+		(property "Datasheet" "~"
+			(at 245.11 74.93 0)
+			(effects
+				(font
+					(size 1.27 1.27)
+				)
+				(hide yes)
+			)
+		)
+		(property "Description" "Light emitting diode"
+			(at 245.11 74.93 0)
+			(effects
+				(font
+					(size 1.27 1.27)
+				)
+				(hide yes)
+			)
+		)
+		(property "Sim.Pins" "1=K 2=A"
+			(at 245.11 74.93 0)
+			(effects
+				(font
+					(size 1.27 1.27)
+				)
+				(hide yes)
+			)
+		)
+		(pin "1"
+		)
+		(pin "2"
+		)
+		(instances
+			(project "moog_prodigy_project"
+				(path "/db469bdb-b6c3-4a16-9199-d4e6b8d556e8/632a0a15-d2db-46b0-8553-670bc8b18225"
+					(reference "D7")
+					(unit 1)
+				)
+			)
+		)
 	)
 	(symbol
@@
 	)
 	(symbol
-		(lib_id "Device:LED")
-		(at 245.11 74.93 90)
-		(unit 1)
-		(exclude_from_sim no)
-		(in_bom yes)
-		(on_board yes)
-		(dnp no)
-		(property "Reference" "D7"
-			(at 241.808 72.39 90)
-			(effects
-				(font
-					(size 1.27 1.27)
-				)
-				(justify right)
-			)
-		)
-		(property "Value" "RED LED"
-			(at 245.872 81.026 90)
-			(effects
-				(font
-					(size 1.27 1.27)
-				)
-				(justify right)
-			)
-		)
-		(property "Footprint" ""
-			(at 245.11 74.93 0)
-			(effects
-				(font
-					(size 1.27 1.27)
-				)
-				(hide yes)
-			)
-		)
-		(property "Datasheet" "~"
-			(at 245.11 74.93 0)
-			(effects
-				(font
-					(size 1.27 1.27)
-				)
-				(hide yes)
-			)
-		)
-		(property "Description" "Light emitting diode"
-			(at 245.11 74.93 0)
-			(effects
-				(font
-					(size 1.27 1.27)
-				)
-				(hide yes)
-			)
-		)
-		(property "Sim.Pins" "1=K 2=A"
-			(at 245.11 74.93 0)
-			(effects
-				(font
-					(size 1.27 1.27)
-				)
-				(hide yes)
-			)
-		)
-		(pin "1"
-		)
-		(pin "2"
-		)
-		(instances
-			(project "moog_prodigy_project"
-				(path "/db469bdb-b6c3-4a16-9199-d4e6b8d556e8/632a0a15-d2db-46b0-8553-670bc8b18225"
-					(reference "D7")
-					(unit 1)
-				)
-			)
-		)
-	)
-	(symbol
 		(lib_id "Device:C_Small")
 		(at 190.5 76.2 0)
@@
 			)
 		)
-		(property "Value" "230 VAC/ 15VAC 1.5A 22W"
+		(property "Value" "230 VAC/ 15VAC 1A5 22W"
 			(at 93.726 31.242 0)
 			(effects
@@
 	)
 	(symbol
+		(lib_name "LED_1")
 		(lib_id "Device:LED")
 		(at 245.11 40.64 270)

Commit message: treba mi da preraspodelim CA 3046
Connections:
- net +12V: now also D6.2 (A); no longer D6.1 (K)
- net at R115.1: now also D6.1 (K); no longer D6.2 (A)
Other:
- moved on the sheet: D6
Changed lines of the file:
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@@
 		(dnp no)
 		(property "Reference" "U24"
-			(at 205.74 24.8412 0)
+			(at 205.486 25.908 0)
 			(effects
 				(font
@@
 		)
 		(property "Value" "LM78L12"
-			(at 205.74 27.3812 0)
+			(at 205.486 28.448 0)
 			(effects
 				(font
@@
 		)
 		(instances
-			(project ""
+			(project "moog_prodigy_project"
 				(path "/db469bdb-b6c3-4a16-9199-d4e6b8d556e8/632a0a15-d2db-46b0-8553-670bc8b18225"
 					(reference "#PWR0142")
@@
 		(dnp no)
 		(property "Reference" "U25"
-			(at 205.74 90.7288 0)
+			(at 205.74 90.9828 0)
 			(effects
 				(font
@@
 		)
 		(property "Value" "LM79L12"
-			(at 205.74 88.1888 0)
+			(at 205.74 88.4428 0)
 			(effects
 				(font
@@
 		(dnp no)
 		(property "Reference" "D7"
-			(at 249.682 75.438 90)
+			(at 243.078 69.85 90)
 			(effects
 				(font
@@
 		)
 		(property "Value" "RED LED"
-			(at 253.492 80.772 90)
+			(at 244.602 72.136 90)
 			(effects
 				(font
@@
 		)
 		(instances
-			(project ""
+			(project "moog_prodigy_project"
 				(path "/db469bdb-b6c3-4a16-9199-d4e6b8d556e8/632a0a15-d2db-46b0-8553-670bc8b18225"
 					(reference "R115")
@@
 		)
 		(instances
-			(project ""
+			(project "moog_prodigy_project"
 				(path "/db469bdb-b6c3-4a16-9199-d4e6b8d556e8/632a0a15-d2db-46b0-8553-670bc8b18225"
 					(reference "T2")
@@
 		(lib_name "LED_1")
 		(lib_id "Device:LED")
-		(at 245.11 40.64 270)
+		(at 245.11 40.64 90)
 		(unit 1)
 		(exclude_from_sim no)
@@
 		(dnp no)
 		(property "Reference" "D6"
-			(at 247.142 39.116 90)
+			(at 241.554 36.068 90)
 			(effects
 				(font
@@
 		)
 		(property "Value" "RED LED"
-			(at 245.872 43.434 90)
+			(at 244.348 37.846 90)
 			(effects
 				(font
@@
 		)
 		(instances
-			(project ""
+			(project "moog_prodigy_project"
 				(path "/db469bdb-b6c3-4a16-9199-d4e6b8d556e8/632a0a15-d2db-46b0-8553-670bc8b18225"
 					(reference "D6")

Commit message: 04.07.2026 Dodati tolerancije, E94, prosiriti spisak
Parts:
- D6, D7: value RED LED -> RED
- F1: value T125mA (spori) -> T125mA (slow)
- F2, F3: value T 1A (brzi) -> T 1A (fast)
Other:
- note added: "AC main supply"
- note removed: "Napajanje iz mreže"
Changed lines of the file:
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@@
 		(comment 4 "Miodrag Babić E1 87/2023")
 	)
-	(text "Napajanje\niz mreže"
+	(text "AC main\nsupply"
 		(exclude_from_sim no)
-		(at 45.974 42.164 0)
+		(at 46.736 42.164 0)
 		(effects
 			(font
 				(size 1.27 1.27)
+				(thickness 0.254)
+				(bold yes)
 			)
 		)
@@
 	(wire
 		(pts
-			(xy 166.37 31.75) (xy 166.37 41.91)
+			(xy 165.1 31.75) (xy 165.1 41.91)
 		)
 		(stroke
@@
 	(wire
 		(pts
-			(xy 166.37 31.75) (xy 173.99 31.75)
+			(xy 165.1 31.75) (xy 173.99 31.75)
 		)
 		(stroke
@@
 	(wire
 		(pts
-			(xy 166.37 41.91) (xy 163.83 41.91)
+			(xy 165.1 41.91) (xy 163.83 41.91)
 		)
 		(stroke
@@
 		(dnp no)
 		(property "Reference" "CP10"
-			(at 256.54 73.66 0)
+			(at 254 73.66 0)
 			(effects
 				(font
@@
 		)
 		(property "Value" "10u"
-			(at 262.9916 76.708 0)
+			(at 253.5428 75.8698 0)
 			(effects
 				(font
@@
 		)
 		(property "Rated Voltage" "25V"
-			(at 260.9088 78.5622 0)
+			(at 251.46 77.724 0)
 			(effects
 				(font
@@
 		(dnp no)
 		(property "Reference" "CP7"
-			(at 172.974 37.846 0)
+			(at 170.942 39.878 0)
 			(effects
 				(font
@@
 		)
 		(property "Value" "2200u"
-			(at 182.372 40.132 0)
+			(at 172.72 42.418 0)
 			(effects
 				(font
@@
 		)
 		(property "Rated Voltage" "25V"
-			(at 178.562 42.418 0)
+			(at 168.91 44.704 0)
 			(effects
 				(font
@@
 		(dnp no)
 		(property "Reference" "D7"
-			(at 243.078 69.85 90)
+			(at 241.808 73.152 90)
 			(effects
 				(font
@@
 			)
 		)
-		(property "Value" "RED LED"
-			(at 244.602 72.136 90)
+		(property "Value" "RED"
+			(at 242.57 75.438 90)
 			(effects
 				(font
@@
 		(on_board yes)
 		(dnp no)
-		(fields_autoplaced yes)
 		(property "Reference" "R115"
-			(at 247.65 48.2599 0)
+			(at 238.252 48.514 0)
 			(effects
 				(font
@@
 		)
 		(property "Value" "1K"
-			(at 247.65 50.7999 0)
+			(at 238.252 51.054 0)
 			(effects
 				(font
@@
 		(dnp no)
 		(property "Reference" "D4"
-			(at 234.696 41.148 90)
+			(at 226.06 41.148 90)
 			(effects
 				(font
@@
 		)
 		(property "Value" "1N4001"
-			(at 232.664 43.434 90)
+			(at 224.028 43.434 90)
 			(effects
 				(font
@@
 		(on_board yes)
 		(dnp no)
-		(fields_autoplaced yes)
 		(property "Reference" "C33"
-			(at 193.04 39.3762 0)
+			(at 184.404 39.624 0)
 			(effects
 				(font
@@
 		)
 		(property "Value" "100n"
-			(at 193.04 41.9162 0)
+			(at 184.404 42.164 0)
 			(effects
 				(font
@@
 		(on_board yes)
 		(dnp no)
-		(fields_autoplaced yes)
 		(property "Reference" "C34"
-			(at 193.04 74.9362 0)
+			(at 183.896 74.93 0)
 			(effects
 				(font
@@
 		)
 		(property "Value" "100n"
-			(at 193.04 77.4762 0)
+			(at 183.896 77.47 0)
 			(effects
 				(font
@@
 			)
 		)
-		(property "Value" "T125mA (spori)"
+		(property "Value" "T125mA (slow)"
 			(at 79.502 36.83 90)
 			(effects
@@
 		(on_board yes)
 		(dnp no)
-		(fields_autoplaced yes)
 		(property "Reference" "C36"
-			(at 222.25 73.6662 0)
+			(at 212.598 73.914 0)
 			(effects
 				(font
@@
 		)
 		(property "Value" "100n"
-			(at 222.25 76.2062 0)
+			(at 212.598 76.454 0)
 			(effects
 				(font
@@
 		(on_board yes)
 		(dnp no)
-		(fields_autoplaced yes)
 		(property "Reference" "C35"
-			(at 222.25 39.3762 0)
+			(at 211.836 39.878 0)
 			(effects
 				(font
@@
 		)
 		(property "Value" "100n"
-			(at 222.25 41.9162 0)
+			(at 211.836 42.418 0)
 			(effects
 				(font
@@
 			)
 		)
-		(property "Value" "T 1A (brzi)"
+		(property "Value" "T 1A (fast)"
 			(at 125.73 53.34 90)
 			(effects
@@
 		(dnp no)
 		(property "Reference" "D5"
-			(at 234.95 75.438 90)
+			(at 226.568 75.184 90)
 			(effects
 				(font
@@
 		)
 		(property "Value" "1N4001"
-			(at 232.664 77.724 90)
+			(at 224.282 77.47 90)
 			(effects
 				(font
@@
 		(dnp no)
 		(property "Reference" "CP8"
-			(at 172.974 73.152 0)
+			(at 168.91 73.152 0)
 			(effects
 				(font
@@
 		)
 		(property "Value" "2200u"
-			(at 182.626 73.914 0)
+			(at 171.45 75.438 0)
 			(effects
 				(font
@@
 		)
 		(property "Rated Voltage" "25V"
-			(at 178.054 76.2 0)
+			(at 166.878 77.724 0)
 			(effects
 				(font
@@
 			)
 		)
-		(property "Value" "T 1A (brzi)"
+		(property "Value" "T 1A (fast)"
 			(at 124.46 30.48 90)
 			(effects
@@
 		(on_board yes)
 		(dnp no)
-		(fields_autoplaced yes)
 		(property "Reference" "R116"
-			(at 247.65 63.4999 0)
+			(at 238.76 63.5 0)
 			(effects
 				(font
@@
 		)
 		(property "Value" "1K"
-			(at 247.65 66.0399 0)
+			(at 238.76 66.04 0)
 			(effects
 				(font
@@
 		(dnp no)
 		(property "Reference" "CP9"
-			(at 256.032 38.862 0)
+			(at 254 40.132 0)
 			(effects
 				(font
@@
 		)
 		(property "Value" "10u"
-			(at 262.9916 41.148 0)
+			(at 255.0668 43.1038 0)
 			(effects
 				(font
@@
 		)
 		(property "Rated Voltage" "25V"
-			(at 260.9088 43.0022 0)
+			(at 252.984 44.958 0)
 			(effects
 				(font
@@
 		(dnp no)
 		(property "Reference" "D6"
-			(at 241.554 36.068 90)
+			(at 241.3 39.624 90)
 			(effects
 				(font
@@
 			)
 		)
-		(property "Value" "RED LED"
-			(at 244.348 37.846 90)
+		(property "Value" "RED"
+			(at 242.316 41.91 90)
 			(effects
 				(font

Commit message: 07.06.2026 fix 3
Parts:
- removed D7: RED, symbol Device:LED
- removed R116: 1K, symbol Device:R
- added D10: RED, symbol Device:LED
- added R32: 330 5%, symbol Device:R
- C10: renamed from CP10; value 10u -> 10u/25V
- C7: renamed from CP7; value 2200u -> 1000u/35V; Rated Voltage 25V -> 35V
- C8: renamed from CP8; value 2200u -> 1000u/35V; Rated Voltage 25V -> 35V
- C9: renamed from CP9; value 10u -> 10u/25V
- F1: value T125mA (slow) -> 125mA/T
- F2, F3: value T 1A (fast) -> 1A/F
- R115: value 1K -> 330 5%
- U24: value LM78L12 -> LM7812
- U25: value LM79L12 -> LM7912
- renumbered ON/OFF1 to SW1_0
Connections:
- net +12V: now also D10.2 (A); no longer D6.2 (A)
- net -12V: now also D6.2 (A)
- net GND: now also R32.2; no longer D1.4, F3.2
- new net: D1.4, F3.2
- new net: D10.1 (K), R32.1
Other:
- note added: "ON OFF"
- moved on the sheet: C10, C33, C34, C35, C36, C7, C8, C9, D1, D2, D3, D4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

Commit message: CA3046 nova schema
Connections:
- net -12V: now also D6.1 (K); no longer D6.2 (A)
- net at R115.1: now also D6.2 (A); no longer D6.1 (K)
Other:
- note added: "NAPOMENA 1 Kondenzatori koji moraju biti kvalitetni: C7,C8,C9,C10,C33,C34,C35,C36"
- moved on the sheet: D6
Changed lines of the file:
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@@
+		)
+	)
+	(text "NAPOMENA 1\nKondenzatori koji moraju biti kvalitetni:\nC7,C8,C9,C10,C33,C34,C35,C36"
+		(exclude_from_sim no)
+		(at 181.356 159.512 0)
+		(effects
+			(font
+				(size 1.27 1.27)
+				(thickness 0.254)
+				(bold yes)
+			)
+			(justify left)
 		)
 	)
@@
 	(wire
 		(pts
+			(xy 237.49 86.36) (xy 237.49 87.63)
+		)
+		(stroke
+			(width 0)
+			(type default)
+		)
+	)
+	(wire
+		(pts
 			(xy 250.19 72.39) (xy 250.19 76.2)
 		)
@@
 	(wire
 		(pts
+			(xy 123.19 34.29) (xy 129.54 34.29)
+		)
+		(stroke
+			(width 0)
+			(type default)
+		)
+	)
+	(wire
+		(pts
+			(xy 214.63 31.75) (xy 224.79 31.75)
+		)
+		(stroke
+			(width 0)
+			(type default)
+		)
+	)
+	(wire
+		(pts
+			(xy 214.63 86.36) (xy 224.79 86.36)
+		)
+		(stroke
+			(width 0)
+			(type default)
+		)
+	)
+	(wire
+		(pts
+			(xy 179.07 41.91) (xy 179.07 48.26)
+		)
+		(stroke
+			(width 0)
+			(type default)
+		)
+	)
+	(wire
+		(pts
+			(xy 224.79 69.85) (xy 224.79 76.2)
+		)
+		(stroke
+			(width 0)
+			(type default)
+		)
+	)
+	(wire
+		(pts
+			(xy 171.45 41.91) (xy 179.07 41.91)
+		)
+		(stroke
+			(width 0)
+			(type default)
+		)
+	)
+	(wire
+		(pts
+			(xy 146.05 44.45) (xy 146.05 76.2)
+		)
+		(stroke
+			(width 0)
+			(type default)
+		)
+	)
+	(wire
+		(pts
+			(xy 224.79 41.91) (xy 218.44 41.91)
+		)
+		(stroke
+			(width 0)
+			(type default)
+		)
+	)
+	(wire
+		(pts
+			(xy 207.01 31.75) (xy 195.58 31.75)
+		)
+		(stroke
+			(width 0)
+			(type default)
+		)
+	)
+	(wire
+		(pts
+			(xy 156.21 34.29) (xy 156.21 36.83)
+		)
+		(stroke
+			(width 0)
+			(type default)
+		)
+	)
+	(wire
+		(pts
+			(xy 224.79 53.34) (xy 224.79 59.69)
+		)
+		(stroke
+			(width 0)
+			(type default)
+		)
+	)
+	(wire
+		(pts
+			(xy 195.58 76.2) (xy 203.2 76.2)
+		)
+		(stroke
+			(width 0)
+			(type default)
+		)
+	)
+	(wire
+		(pts
+			(xy 237.49 41.91) (xy 224.79 41.91)
+		)
+		(stroke
+			(width 0)
+			(type default)
+		)
+	)
+	(wire
+		(pts
+			(xy 203.2 41.91) (xy 195.58 41.91)
+		)
+		(stroke
+			(width 0)
+			(type default)
+		)
+	)
+	(wire
+		(pts
+			(xy 224.79 59.69) (xy 237.49 59.69)
+		)
+		(stroke
+			(width 0)
+			(type default)
+		)
+	)
+	(wire
+		(pts
+			(xy 64.77 36.83) (xy 72.39 36.83)
+		)
+		(stroke
+			(width 0)
+			(type default)
+		)
+	)
+	(wire
+		(pts
+			(xy 224.79 31.75) (xy 224.79 41.91)
+		)
+		(stroke
+			(width 0)
+			(type default)
+		)
+	)
+	(wire
+		(pts
+			(xy 124.46 41.91) (xy 123.19 41.91)
+		)
+		(stroke
+			(width 0)
+			(type default)
+		)
+	)
+	(wire
+		(pts
+			(xy 128.27 44.45) (xy 128.27 59.69)
+		)
+		(stroke
+			(width 0)
+			(type default)
+		)
+	)
+	(wire
+		(pts
+			(xy 64.77 46.99) (xy 72.39 46.99)
+		)
+		(stroke
+			(width 0)
+			(type default)
+		)
+	)
+	(wire
+		(pts
+			(xy 207.01 86.36) (xy 195.58 86.36)
+		)
+		(stroke
+			(width 0)
+			(type default)
+		)
+	)
+	(wire
+		(pts
 			(xy 237.49 76.2) (xy 237.49 78.74)
-		)
-		(stroke
-			(width 0)
-			(type default)
-		)
-	)
-	(wire
-		(pts
-			(xy 123.19 34.29) (xy 129.54 34.29)
-		)
-		(stroke
-			(width 0)
-			(type default)
-		)
-	)
-	(wire
-		(pts
-			(xy 214.63 31.75) (xy 224.79 31.75)
-		)
-		(stroke
-			(width 0)
-			(type default)
-		)
-	)
-	(wire
-		(pts
-			(xy 237.49 86.36) (xy 237.49 87.63)
-		)
-		(stroke
-			(width 0)
-			(type default)
-		)
-	)
-	(wire
-		(pts
-			(xy 214.63 86.36) (xy 224.79 86.36)
-		)
-		(stroke
-			(width 0)
-			(type default)
-		)
-	)
-	(wire
-		(pts
-			(xy 179.07 41.91) (xy 179.07 48.26)
-		)
-		(stroke
-			(width 0)
-			(type default)
-		)
-	)
-	(wire
-		(pts
-			(xy 224.79 69.85) (xy 224.79 76.2)
-		)
-		(stroke
-			(width 0)
-			(type default)
-		)
-	)
-	(wire
-		(pts
-			(xy 171.45 41.91) (xy 179.07 41.91)
-		)
-		(stroke
-			(width 0)
-			(type default)
-		)
-	)
-	(wire
-		(pts
-			(xy 146.05 44.45) (xy 146.05 76.2)
-		)
-		(stroke
-			(width 0)
-			(type default)
-		)
-	)
-	(wire
-		(pts
-			(xy 224.79 41.91) (xy 218.44 41.91)
-		)
-		(stroke
-			(width 0)
-			(type default)
-		)
-	)
-	(wire
-		(pts
-			(xy 207.01 31.75) (xy 195.58 31.75)
-		)
-		(stroke
-			(width 0)
-			(type default)
-		)
-	)
-	(wire
-		(pts
-			(xy 156.21 34.29) (xy 156.21 36.83)
-		)
-		(stroke
-			(width 0)
-			(type default)
-		)
-	)
-	(wire
-		(pts
-			(xy 224.79 53.34) (xy 224.79 59.69)
-		)
-		(stroke
-			(width 0)
-			(type default)
-		)
-	)
-	(wire
-		(pts
-			(xy 195.58 76.2) (xy 203.2 76.2)
-		)
-		(stroke
-			(width 0)
-			(type default)
-		)
-	)
-	(wire
-		(pts
-			(xy 237.49 41.91) (xy 224.79 41.91)
-		)
-		(stroke
-			(width 0)
-			(type default)
-		)
-	)
-	(wire
-		(pts
-			(xy 203.2 41.91) (xy 195.58 41.91)
-		)
-		(stroke
-			(width 0)
-			(type default)
-		)
-	)
-	(wire
-		(pts
-			(xy 224.79 59.69) (xy 237.49 59.69)
-		)
-		(stroke
-			(width 0)
-			(type default)
-		)
-	)
-	(wire
-		(pts
-			(xy 64.77 36.83) (xy 72.39 36.83)
-		)
-		(stroke
-			(width 0)
-			(type default)
-		)
-	)
-	(wire
-		(pts
-			(xy 224.79 31.75) (xy 224.79 41.91)
-		)
-		(stroke
-			(width 0)
-			(type default)
-		)
-	)
-	(wire
-		(pts
-			(xy 124.46 41.91) (xy 123.19 41.91)
-		)
-		(stroke
-			(width 0)
-			(type default)
-		)
-	)
-	(wire
-		(pts
-			(xy 128.27 44.45) (xy 128.27 59.69)
-		)
-		(stroke
-			(width 0)
-			(type default)
-		)
-	)
-	(wire
-		(pts
-			(xy 64.77 46.99) (xy 72.39 46.99)
-		)
-		(stroke
-			(width 0)
-			(type default)
-		)
-	)
-	(wire
-		(pts
-			(xy 207.01 86.36) (xy 195.58 86.36)
 		)
 		(stroke
@@
 		(lib_name "LED_1")
 		(lib_id "Device:LED")
-		(at 237.49 82.55 90)
+		(at 237.49 82.55 270)
 		(unit 1)
 		(exclude_from_sim no)
@@
 		(dnp no)
 		(property "Reference" "D6"
-			(at 234.442 81.534 90)
+			(at 240.538 83.566 90)
 			(effects
 				(font
@@
 		)
 		(property "Value" "RED"
-			(at 234.696 83.82 90)
-			(effects
-				(font
+			(at 240.284 81.28 90)
+			(effects
+				(font

Commit message: 08.07.2026 fix
Parts:
- renumbered C7 to C44, C8 to C45, C9 to C46, C10 to C47
Other:
- note removed: "NAPOMENA 1 Kondenzatori koji moraju biti kvalitetni: C7,C8,C9,C10,C33,C34,C35,C36"
- moved on the sheet: C47, F2
Changed lines of the file:
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@@
 		)
 	)
-	(text "NAPOMENA 1\nKondenzatori koji moraju biti kvalitetni:\nC7,C8,C9,C10,C33,C34,C35,C36"
-		(exclude_from_sim no)
-		(at 181.356 159.512 0)
-		(effects
-			(font
-				(size 1.27 1.27)
-				(thickness 0.254)
-				(bold yes)
-			)
-			(justify left)
-		)
-	)
 	(text "AC main\nsupply"
 		(exclude_from_sim no)
@@
 	(wire
 		(pts
-			(xy 156.21 34.29) (xy 137.16 34.29)
+			(xy 156.21 34.29) (xy 138.43 34.29)
 		)
 		(stroke
@@
 	(wire
 		(pts
-			(xy 250.19 72.39) (xy 250.19 76.2)
+			(xy 250.19 71.12) (xy 250.19 76.2)
 		)
 		(stroke
@@
 	(wire
 		(pts
-			(xy 250.19 59.69) (xy 250.19 66.04)
+			(xy 250.19 59.69) (xy 250.19 64.77)
 		)
 		(stroke
@@
 	(wire
 		(pts
-			(xy 123.19 34.29) (xy 129.54 34.29)
+			(xy 123.19 34.29) (xy 130.81 34.29)
 		)
 		(stroke
@@
 		(lib_name "elektrolit_3")
 		(lib_id "elektrolitski:elektrolit")
-		(at 250.19 68.58 0)
+		(at 250.19 67.31 0)
 		(unit 1)
 		(exclude_from_sim no)
@@
 		(on_board yes)
 		(dnp no)
-		(property "Reference" "C10"
-			(at 247.142 68.326 0)
+		(property "Reference" "C47"
+			(at 247.142 67.056 0)
 			(effects
 				(font
@@
 		)
 		(property "Value" "10u/25V"
-			(at 249.682 71.12 0)
+			(at 249.682 69.85 0)
 			(effects
 				(font
@@
 		)
 		(property "Footprint" "Capacitor_THT:CP_Radial_D5.0mm_P2.50mm"
-			(at 250.19 80.01 0)
+			(at 250.19 78.74 0)
 			(effects
 				(font
@@
 		)
 		(property "Datasheet" ""
-			(at 249.936 68.58 0)
+			(at 249.936 67.31 0)
 			(effects
 				(font
@@
 		)
 		(property "Description" ""
-			(at 250.19 68.58 0)
+			(at 250.19 67.31 0)
 			(effects
 				(font
@@
 		)
 		(property "Rated Voltage" "25V"
-			(at 245.11 70.104 0)
+			(at 245.11 68.834 0)
 			(effects
 				(font
@@
 			(project "moog_prodigy_project"
 				(path "/db469bdb-b6c3-4a16-9199-d4e6b8d556e8/632a0a15-d2db-46b0-8553-670bc8b18225"
-					(reference "C10")
+					(reference "C47")
 					(unit 1)
 				)
@@
 		(on_board yes)
 		(dnp no)
-		(property "Reference" "C7"
+		(property "Reference" "C44"
 			(at 174.498 50.8 0)
 			(effects
@@
 			(project "moog_prodigy_project"
 				(path "/db469bdb-b6c3-4a16-9199-d4e6b8d556e8/632a0a15-d2db-46b0-8553-670bc8b18225"
-					(reference "C7")
+					(reference "C44")
 					(unit 1)
 				)
@@
 		(dnp no)
 		(property "Reference" "R32"
-			(at 264.16 58.674 0)
+			(at 263.398 58.928 0)
 			(effects
 				(font
@@
 		)
 		(property "Value" "330 5%"
-			(at 261.874 61.214 0)
+			(at 261.366 61.214 0)
 			(effects
 				(font
@@
 		(on_board yes)
 		(dnp no)
-		(property "Reference" "C8"
+		(property "Reference" "C45"
 			(at 174.244 66.802 0)
 			(effects
@@
 			(project "moog_prodigy_project"
 				(path "/db469bdb-b6c3-4a16-9199-d4e6b8d556e8/632a0a15-d2db-46b0-8553-670bc8b18225"
-					(reference "C8")
+					(reference "C45")
 					(unit 1)
 				)
@@
 	(symbol
 		(lib_id "Device:Fuse")
-		(at 133.35 34.29 90)
+		(at 134.62 34.29 90)
 		(unit 1)
 		(exclude_from_sim no)
@@
 		(fields_autoplaced yes)
 		(property "Reference" "F2"
-			(at 133.35 27.94 90)
+			(at 134.62 27.94 90)
 			(effects
 				(font
@@
 		)
 		(property "Value" "1A/F"
-			(at 133.35 30.48 90)
+			(at 134.62 30.48 90)
 			(effects
 				(font
@@
 		)
 		(property "Footprint" "Fuse:Fuse_Bourns_MF-RHT100"
-			(at 133.35 36.068 90)
+			(at 134.62 36.068 90)
 			(effects
 				(font
@@
 		)
 		(property "Datasheet" "~"
-			(at 133.35 34.29 0)
+			(at 134.62 34.29 0)
 			(effects
 				(font
@@
 		)
 		(property "Description" ""
-			(at 133.35 34.29 0)
+			(at 134.62 34.29 0)
 			(effects
 				(font
@@
 		(on_board yes)
 		(dnp no)
-		(property "Reference" "C9"
+		(property "Reference" "C46"
 			(at 246.888 50.8 0)
 			(effects
@@
 			(project "moog_prodigy_project"
 				(path "/db469bdb-b6c3-4a16-9199-d4e6b8d556e8/632a0a15-d2db-46b0-8553-670bc8b18225"
-					(reference "C9")
+					(reference "C46")
 					(unit 1)
 				)
