File: Moog_Prodigy_Project/moog_prodigy_project/voltage_source.kicad_sch (KiCad schematic)
At the start: 24 parts, among them SW1_0 200MDP1T1B1M2QEH, T2 230 VAC/ 15VAC 1A5 22W, U24 LM7812, U25 LM7912

Commit message: Finalni deo seme, prelaz na PCB
Parts:
- T2: value 230 VAC/ 15VAC 1A5 22W -> 230VAC / 2x15VAC 0A53 16VA; footprint Transformer_THT:Transformer_Myrra_EI30-5_44000_Horizontal -> Transformer_THT:Transformer_CHK_EI54-16VA_2xSec
- renumbered C44 to C94, C45 to C95, C46 to C96, C47 to C97, R32 to R153
Other:
- note added: "*GENERAL NOTE* Resistor values that are not explicitly specified are selected from the E96 value series with a tolerance of ±1%."
Changed lines of the file:
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@@
 		)
 	)
+	(text "*GENERAL NOTE*\nResistor values that are not explicitly specified\nare selected from the E96 value series with a \ntolerance of ±1%."
+		(exclude_from_sim no)
+		(at 177.038 159.512 0)
+		(effects
+			(font
+				(size 1.27 1.27)
+				(thickness 0.254)
+				(bold yes)
+			)
+			(justify left)
+		)
+	)
 	(junction
 		(at 124.46 44.45)
@@
 		(on_board yes)
 		(dnp no)
-		(property "Reference" "#PWR?"
+		(property "Reference" "#PWR0117"
 			(at 270.51 69.85 0)
 			(effects
@@
 			(project "moog_prodigy_project"
 				(path "/db469bdb-b6c3-4a16-9199-d4e6b8d556e8/632a0a15-d2db-46b0-8553-670bc8b18225"
-					(reference "#PWR?")
+					(reference "#PWR0117")
 					(unit 1)
 				)
@@
 		(on_board yes)
 		(dnp no)
-		(property "Reference" "C47"
+		(property "Reference" "C97"
 			(at 247.142 67.056 0)
 			(effects
@@
 			(project "moog_prodigy_project"
 				(path "/db469bdb-b6c3-4a16-9199-d4e6b8d556e8/632a0a15-d2db-46b0-8553-670bc8b18225"
-					(reference "C47")
+					(reference "C97")
 					(unit 1)
 				)
@@
 		(on_board yes)
 		(dnp no)
-		(property "Reference" "C44"
+		(property "Reference" "C94"
 			(at 174.498 50.8 0)
 			(effects
@@
 			(project "moog_prodigy_project"
 				(path "/db469bdb-b6c3-4a16-9199-d4e6b8d556e8/632a0a15-d2db-46b0-8553-670bc8b18225"
-					(reference "C44")
+					(reference "C94")
 					(unit 1)
 				)
@@
 		(on_board yes)
 		(dnp no)
-		(property "Reference" "R32"
+		(property "Reference" "R153"
 			(at 263.398 58.928 0)
 			(effects
@@
 			(project "moog_prodigy_project"
 				(path "/db469bdb-b6c3-4a16-9199-d4e6b8d556e8/632a0a15-d2db-46b0-8553-670bc8b18225"
-					(reference "R32")
+					(reference "R153")
 					(unit 1)
 				)
@@
 			)
 		)
-		(property "Value" "230 VAC/ 15VAC 1A5 22W"
+		(property "Value" "230VAC / 2x15VAC 0A53 16VA"
 			(at 112.776 31.242 0)
 			(effects
@@
 			)
 		)
-		(property "Footprint" "Transformer_THT:Transformer_Myrra_EI30-5_44000_Horizontal"
+		(property "Footprint" "Transformer_THT:Transformer_CHK_EI54-16VA_2xSec"
 			(at 113.03 44.45 0)
 			(effects
@@
 		(on_board yes)
 		(dnp no)
-		(property "Reference" "C45"
+		(property "Reference" "C95"
 			(at 174.244 66.802 0)
 			(effects
@@
 			(project "moog_prodigy_project"
 				(path "/db469bdb-b6c3-4a16-9199-d4e6b8d556e8/632a0a15-d2db-46b0-8553-670bc8b18225"
-					(reference "C45")
+					(reference "C95")
 					(unit 1)
 				)
@@
 		(on_board yes)
 		(dnp no)
-		(property "Reference" "C46"
+		(property "Reference" "C96"
 			(at 246.888 50.8 0)
 			(effects
@@
 			(project "moog_prodigy_project"
 				(path "/db469bdb-b6c3-4a16-9199-d4e6b8d556e8/632a0a15-d2db-46b0-8553-670bc8b18225"
-					(reference "C46")
+					(reference "C96")
 					(unit 1)
 				)
