File: Moog_Prodigy_Project/moog_prodigy_project/4007_mosfets.kicad_sch (KiCad schematic)
At the start: 49 parts, among them Q20 BC327, Q21 BC327, SW12 FINAL DECAY SWITCH, SW13 FINAL DECAY SWITCH, U20 NE556N, U21 MC14007UBCP, U22 MC14007UBCP, U23 MC14007UBCP, U26 OPA184, U27 OPA184

Commit message: treba mi da preraspodelim CA 3046
Connections:
- net THRESHOLD_2: now also C31.2
- net at U22.10, U22.5: now also R137.1; no longer R137.2
- net at U22.12: now also C32.1
- net at U21.10, U22.13, U22.8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: now also R137.2; no longer R137.1
- net at U20.10 (2RESET), U20.4 (1RESET): no longer C31.2
Other:
- note added: "FINAL DECAY SWITCH"
- moved on the sheet: C31, C32, C79, C80, C81, C82, C83, C84, C85, C86, CP11, CP12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

Commit message: 04.07.2026 Dodati tolerancije, E94, prosiriti spisak
Parts:
- Q20, Q21: value BC327 -> BC549
- renumbered RV25 to RV25_LOG, RV26 to RV26_LOG, RV27 to RV27_LOG, RV29 to RV29_LIN, RV30 to RV30_LIN
Connections:
- no-connect marks 10 -> 9
Other:
- moved on the sheet: C81, C82, C83, C84, C85, CP11, CP5, R126, U20, U26

Commit message: 07.06.2026 fix 3
Parts:
- CP11, CP12: value 6u8 -> 6u8/20V
- CP5: value 10u -> 10u/16V
- R147, R151: value 4K3 -> 4K32
- R149: value 56K -> 56K2
Other:
- note added: "NAPOMENA 1 Kondenzatori: C79,C80,C81,C82,C83,C84,C85 su vrednosti 100n i oni su kvalitetniji"
- note removed: "NAPOMENA 1 Kondenzatori: C79,C80,C81,C82,C83,C84,C85 su vrednosti 100n i oni su kvalitetniji Ponteciometri: Linearni:RV29,RV30 Logaritamski: RV25,RV26,RV27"
- note removed: "NAPOMENA 2 Otpornici cija je vrednost: 63K4, 18K2, 4K75, 6K81, 51M, 2.4M su otpornici iz E96 serije (1%) Ostali orpotnici su iz serije E24 (5%)"
- moved on the sheet: CP11, CP12, CP5

Commit message: CA3046 nova schema
Other:
- note added: "NAPOMENA 1 Kondenzatori koji moraju biti kvalitetni: C31,C32,C79,C80,C81,C82,C83,C84,C85 CP5,CP11,CP12"
- note removed: "NAPOMENA 1 Kondenzatori: C79,C80,C81,C82,C83,C84,C85 su vrednosti 100n i oni su kvalitetniji"
Changed lines of the file:
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@@
 		)
 	)
-	(text "NAPOMENA 1\nKondenzatori:\nC79,C80,C81,C82,C83,C84,C85\nsu vrednosti 100n i oni su kvalitetniji"
+	(text "NAPOMENA 1\nKondenzatori koji moraju biti kvalitetni:\nC31,C32,C79,C80,C81,C82,C83,C84,C85\nCP5,CP11,CP12\n"
 		(exclude_from_sim no)
 		(at 300.228 242.062 0)
@@
 	(text "VCA\nATTACK"
 		(exclude_from_sim no)
-		(at 154.178 33.02 0)
-		(effects
-			(font
+		(at 154.686 34.036 0)
+		(effects
+			(font

Commit message: 08.07.2026 fix
Parts:
- C41: renamed from CP12; value 6u8/20V -> 6u8/25V
- C42: renamed from CP11; value 6u8/20V -> 6u8/25V
- RV25: renamed from RV25_LOG; value 1M -> 1M LOG
- RV26: renamed from RV26_LOG; value 1M -> 1M LOG
- RV27: renamed from RV27_LOG; value 1M -> 1M LOG
- RV29: renamed from RV29_LIN; value 10K -> 10K LIN
- RV30: renamed from RV30_LIN; value 10K -> 10K LIN
- renumbered CP5 to C43
Other:
- note added: "PP"
- note removed: "NAPOMENA 1 Kondenzatori koji moraju biti kvalitetni: C31,C32,C79,C80,C81,C82,C83,C84,C85 CP5,CP11,CP12"
Changed lines of the file:
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@@
 		)
 	)
-	(text "NAPOMENA 1\nKondenzatori koji moraju biti kvalitetni:\nC31,C32,C79,C80,C81,C82,C83,C84,C85\nCP5,CP11,CP12\n"
-		(exclude_from_sim no)
-		(at 300.228 242.062 0)
-		(effects
-			(font
-				(size 1.27 1.27)
-				(thickness 0.254)
-				(bold yes)
-			)
-			(justify left)
-		)
-	)
 	(text "IC3_2"
 		(exclude_from_sim no)
@@
 	(text "VCF\nATTACK"
 		(exclude_from_sim no)
-		(at 113.284 108.204 0)
+		(at 113.284 107.442 0)
 		(effects
 			(font
@@
 	(text "IC3_5"
 		(exclude_from_sim no)
-		(at 164.592 221.234 0)
+		(at 165.354 220.218 0)
 		(effects
 			(font
@@
 		)
 	)
+	(text "PP"
+		(exclude_from_sim no)
+		(at 211.074 52.324 0)
+		(effects
+			(font
+				(size 1.27 1.27)
+				(thickness 0.254)
+				(bold yes)
+			)
+		)
+	)
 	(text "IC4_6"
 		(exclude_from_sim no)
@@
 	(text "VCF\nDECAY/RELEASE"
 		(exclude_from_sim no)
-		(at 161.29 130.81 0)
+		(at 161.29 129.286 0)
 		(effects
 			(font
@@
 		)
 	)
+	(text "PP"
+		(exclude_from_sim no)
+		(at 94.742 239.014 0)
+		(effects
+			(font
+				(size 1.27 1.27)
+				(thickness 0.254)
+				(bold yes)
+			)
+		)
+	)
 	(text "IC3"
 		(exclude_from_sim no)
@@
 		)
 	)
+	(text "PP"
+		(exclude_from_sim no)
+		(at 168.91 123.19 0)
+		(effects
+			(font
+				(size 1.27 1.27)
+				(thickness 0.254)
+				(bold yes)
+			)
+		)
+	)
 	(text "VCA\nDECAY/RELEASE"
 		(exclude_from_sim no)
@@
 		)
 	)
+	(text "PP"
+		(exclude_from_sim no)
+		(at 159.766 222.758 0)
+		(effects
+			(font
+				(size 1.27 1.27)
+				(thickness 0.254)
+				(bold yes)
+			)
+		)
+	)
 	(text "IC3_3"
 		(exclude_from_sim no)
@@
 	(text "VCA\nATTACK"
 		(exclude_from_sim no)
-		(at 154.686 34.036 0)
+		(at 154.686 33.528 0)
 		(effects
 			(font
@@
 		(on_board yes)
 		(dnp no)
-		(property "Reference" "CP11"
+		(property "Reference" "C42"
 			(at 213.106 46.99 0)
 			(effects
@@
 			)
 		)
-		(property "Value" "6u8/20V"
+		(property "Value" "6u8/25V"
 			(at 215.138 49.53 0)
 			(effects
@@
 			(project "moog_prodigy_project"
 				(path "/db469bdb-b6c3-4a16-9199-d4e6b8d556e8/e87f9916-2112-448f-9f59-6551b8229296"
-					(reference "CP11")
+					(reference "C42")
 					(unit 1)
 				)
@@
 		(on_board yes)
 		(dnp no)
-		(property "Reference" "CP5"
+		(property "Reference" "C43"
 			(at 328.168 100.33 0)
 			(effects
@@
 			(project "moog_prodigy_project"
 				(path "/db469bdb-b6c3-4a16-9199-d4e6b8d556e8/e87f9916-2112-448f-9f59-6551b8229296"
-					(reference "CP5")
+					(reference "C43")
 					(unit 1)
 				)
@@
 		(on_board yes)
 		(dnp no)
-		(property "Reference" "RV26_LOG"
-			(at 112.776 111.506 90)
+		(property "Reference" "RV26"
+			(at 112.776 110.744 90)
 			(effects
 				(font
@@
 			)
 		)
-		(property "Value" "1M"
-			(at 112.776 113.538 90)
+		(property "Value" "1M LOG"
+			(at 112.776 112.776 90)
 			(effects
 				(font
@@
 			(project "moog_prodigy_project"
 				(path "/db469bdb-b6c3-4a16-9199-d4e6b8d556e8/e87f9916-2112-448f-9f59-6551b8229296"
-					(reference "RV26_LOG")
+					(reference "RV26")
 					(unit 1)
 				)
@@
 		(on_board yes)
 		(dnp no)
-		(property "Reference" "RV27_LOG"
-			(at 189.738 48.514 0)
+		(property "Reference" "RV27"
+			(at 190.754 48.514 0)
 			(effects
 				(font
@@
 			)
 		)
-		(property "Value" "1M"
-			(at 193.04 50.546 0)
+		(property "Value" "1M LOG"
+			(at 189.738 50.546 0)
 			(effects
 				(font
@@
 			(project "moog_prodigy_project"
 				(path "/db469bdb-b6c3-4a16-9199-d4e6b8d556e8/e87f9916-2112-448f-9f59-6551b8229296"
-					(reference "RV27_LOG")
+					(reference "RV27")
 					(unit 1)
 				)
@@
 		(on_board yes)
 		(dnp no)
-		(property "Reference" "CP12"
+		(property "Reference" "C41"
 			(at 170.942 117.602 0)
 			(effects
@@
 			)
 		)
-		(property "Value" "6u8/20V"
+		(property "Value" "6u8/25V"
 			(at 172.72 120.396 0)
 			(effects
@@
 			(project "moog_prodigy_project"
 				(path "/db469bdb-b6c3-4a16-9199-d4e6b8d556e8/e87f9916-2112-448f-9f59-6551b8229296"
-					(reference "CP12")
+					(reference "C41")
 					(unit 1)
 				)
@@
 		(on_board yes)
 		(dnp no)
-		(property "Reference" "RV30_LIN"
-			(at 135.128 86.868 0)
+		(property "Reference" "RV30"
+			(at 135.636 86.868 0)
 			(effects
 				(font
@@
 			)
 		)
-		(property "Value" "10K"
-			(at 137.414 88.9 0)
+		(property "Value" "10K LIN"
+			(at 135.128 88.9 0)
 			(effects
 				(font
@@
 			(project "moog_prodigy_project"
 				(path "/db469bdb-b6c3-4a16-9199-d4e6b8d556e8/e87f9916-2112-448f-9f59-6551b8229296"
-					(reference "RV30_LIN")
+					(reference "RV30")
 					(unit 1)
 				)
@@
 		(dnp no)
 		(property "Reference" "C32"
-			(at 158.75 217.932 0)
+			(at 159.258 217.932 0)
 			(effects
 				(font
@@
 		)
 		(property "Value" "10n"
-			(at 159.004 220.218 0)
+			(at 159.512 220.218 0)
 			(effects
 				(font
@@
 		(on_board yes)
 		(dnp no)
-		(property "Reference" "RV25_LOG"
-			(at 154.94 37.592 90)
+		(property "Reference" "RV25"
+			(at 154.94 37.084 90)
 			(effects
 				(font
@@
 			)
 		)
-		(property "Value" "1M"
-			(at 154.94 39.37 90)
+		(property "Value" "1M LOG"
+			(at 154.94 38.862 90)
 			(effects
 				(font
@@
 			(project "moog_prodigy_project"
 				(path "/db469bdb-b6c3-4a16-9199-d4e6b8d556e8/e87f9916-2112-448f-9f59-6551b8229296"
-					(reference "RV25_LOG")
+					(reference "RV25")
 					(unit 1)
 				)
@@
 		(on_board yes)
 		(dnp no)
-		(property "Reference" "RV29_LIN"
-			(at 107.188 163.322 0)
+		(property "Reference" "RV29"
+			(at 107.95 162.814 0)
 			(effects
 				(font
@@
 			)
 		)
-		(property "Value" "10K"
-			(at 109.474 165.354 0)
+		(property "Value" "10K LIN"
+			(at 107.696 165.1 0)
 			(effects
 				(font
@@
 			(project "moog_prodigy_project"
 				(path "/db469bdb-b6c3-4a16-9199-d4e6b8d556e8/e87f9916-2112-448f-9f59-6551b8229296"
-					(reference "RV29_LIN")
+					(reference "RV29")
 					(unit 1)
 				)

Commit message: Finalni deo seme, prelaz na PCB
Parts:
- renumbered C41 to C91, C42 to C92, C43 to C93
Other:
- note added: "*GENERAL NOTE* Resistor values that are not explicitly specified are selected from the E96 value series with a tolerance of ±1%."
Changed lines of the file:
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@@
 		)
 	)
+	(text "*GENERAL NOTE*\nResistor values that are not explicitly specified\nare selected from the E96 value series with a \ntolerance of ±1%."
+		(exclude_from_sim no)
+		(at 299.974 247.142 0)
+		(effects
+			(font
+				(size 1.27 1.27)
+				(thickness 0.254)
+				(bold yes)
+			)
+			(justify left)
+		)
+	)
 	(text "IC5_3"
 		(exclude_from_sim no)
@@
 		(on_board yes)
 		(dnp no)
-		(property "Reference" "C42"
+		(property "Reference" "C92"
 			(at 213.106 46.99 0)
 			(effects
@@
 			(project "moog_prodigy_project"
 				(path "/db469bdb-b6c3-4a16-9199-d4e6b8d556e8/e87f9916-2112-448f-9f59-6551b8229296"
-					(reference "C42")
+					(reference "C92")
 					(unit 1)
 				)
@@
 		(on_board yes)
 		(dnp no)
-		(property "Reference" "C43"
+		(property "Reference" "C93"
 			(at 328.168 100.33 0)
 			(effects
@@
 			(project "moog_prodigy_project"
 				(path "/db469bdb-b6c3-4a16-9199-d4e6b8d556e8/e87f9916-2112-448f-9f59-6551b8229296"
-					(reference "C43")
+					(reference "C93")
 					(unit 1)
 				)
@@
 		(on_board yes)
 		(dnp no)
-		(property "Reference" "C41"
+		(property "Reference" "C91"
 			(at 170.942 117.602 0)
 			(effects
@@
 			(project "moog_prodigy_project"
 				(path "/db469bdb-b6c3-4a16-9199-d4e6b8d556e8/e87f9916-2112-448f-9f59-6551b8229296"
-					(reference "C41")
+					(reference "C91")
 					(unit 1)
 				)
@@
 		(on_board yes)
 		(dnp no)
-		(property "Reference" "+12V"
+		(property "Reference" "#+12V0101"
 			(at 196.85 104.14 0)
 			(effects
@@
 			(project "moog_prodigy_project"
 				(path "/db469bdb-b6c3-4a16-9199-d4e6b8d556e8/e87f9916-2112-448f-9f59-6551b8229296"
-					(reference "+12V")
+					(reference "#+12V0101")
 					(unit 1)
 				)
