File: Moog_Prodigy_Project/moog_prodigy_project/ledder.kicad_sch (KiCad schematic)
At the start: 72 parts, among them J6 NJ2FD-V, Q10 CA3046, Q11 BC327, Q14 BC550C, Q15 BC550C, Q16 BC550C, Q17 BC550C, Q18 BC550C, Q19 BC550C, Q8 BC556, Q9 CA3046, SW11 FILTER MODE, U1 LT1469, U15 LT1469, U16 LT1228, U17 NE5532

Commit message: treba mi da preraspodelim CA 3046
Parts:
- R104: value 6K81 1% -> 6K81; tolerance (none) -> 1%
- R105: value 6K81 1% -> 6K81
Connections:
- net node_6: no longer C26.2, Q10.6, Q9.7
- net node_7: no longer C26.1, Q10.9, Q9.10
- net at Q10.3, R102.2, R108.2: now also Q10.13, R103.2, R105.2, R106.2
- new net: C29.2, Q17. (E), Q18. (E)
- new net: C29.1, Q14. (E), Q15. (E)
- new net: C26.1, Q10.9, Q9.10
- new net: C26.2, Q10.6, Q9.7
Other:
- note added: "SIGNAL OUT"
- moved on the sheet: C27, C28, C29, C30, C72, C73, C74, C75, C76, C77, CP1, CP6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

Commit message: 04.07.2026 Dodati tolerancije, E94, prosiriti spisak
Parts:
- Q11: value BC327 -> BC549
- Q8: value BC556 -> BC549
- U1: value LT1469 -> NE5532
- renumbered RV12 to RV12_LIN, RV14 to RV14_LOG, RV15 to RV15_LIN, RV16 to RV16_LOG, RV22 to RV22_LIN, RV23 to RV23_LIN
Connections:
- new net: C29.2, Q17. (E), Q18. (E)
- new net: C29.1, Q14. (E), Q15. (E)
Other:
- note added: "NAPOMENA 1 Kondenzatori: C71,C72,C73,C74,C75,C76,C77,C78 su vrednosti 100n i oni su kvalitetniji"
- note removed: "NAPOMENA 1 Kondenzatori: C71,C72,C73,C74,C75,C76,C77,C78 su vrednosti 100n i oni su kvalitetniji Ponteciometri: Linearni:RV12,RV15,RV22,RV23 Logaritamski: RV14,RV16"
- moved on the sheet: C25, C26, C27, C28, C29, C30, C71, C72, C73, C74, C75, C76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

Commit message: 07.06.2026 fix 3
Parts:
- added R126_2, R128_3: 2K, Resistor_THT:R_Axial_DIN0207_L6.3mm_D2.5mm_P7.62mm_Horizontal, symbol Device:R
- added R128_2: 10K, Resistor_THT:R_Axial_DIN0207_L6.3mm_D2.5mm_P7.62mm_Horizontal, symbol Device:R
- CP1: value 2u2 -> 2u2/16V
- R126_1: value 51K -> 49K
- R128_1: value 36K -> 34K8
- RV14_LOG: value 50K -> 51K1
Connections:
- net node_2: now also R126_2.2; no longer R126_1.2
- net at R128_1.2: now also R128_2.1; no longer SW11.2 (B)
- new net: C29.2, Q17. (E), Q18. (E)
- new net: C29.1, Q14. (E), Q15. (E)
- new net: R126_1.2, R126_2.1
- new net: R128_2.2, R128_3.1
- new net: R128_3.2, SW11.2 (B)
Other:
- note removed: "NAPOMENA 2 Otpornici cija je vrednost: 63K4, 18K2, 4K75, 6K81, 51M, 2.4M su otpornici iz E96 serije (1%) Ostali orpotnici su iz serije E24 (5%)"
- moved on the sheet: R126_1, R128_1, SW11

Commit message: CA3046 nova schema
Parts:
- removed Q10, Q9: CA3046, CA3046:DIL14, symbol CA3046:CA3046
- added IC1, IC2: 2N3055, Package_TO_SOT_THT:TO-3, symbol Transistor_BJT:2N3055
- added IC1_3, IC1_4, IC1_5, IC2_3, IC2_4, IC2_5: BC550C, Package_TO_SOT_THT:TO-92_Inline, symbol Transistor_BJT:BC550
Connections:
- net node_2 is gone; now on net -12V: Q8. (E), R126_2.2, R127_1.1, R128_1.1, R132.2, R133.2, RV24.3
- net +12V: now also C77.2, IC1.1 (C), IC1_3.8 (C), IC1_4.11 (C), IC2_5.14 (C); no longer C77.1
- net GND: now also C77.1, IC1_5.13; no longer C77.2
- net at R102.2, R103.2, R105.2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: now also IC1.3 (E), IC2_5.13
- net at C26.1: now also IC1_3.7, IC2_3.6 (B)
- net at R96.1: now also IC1_5.14 (C)
- net at CP1., R98.1: now also IC2.2 (B)
- net at R96.2: now also IC2.3 (E)
- net at R100.1, RV13.3: now also CP6., R108_1.1, R131.2, R98.2, R99.2; no longer R99.1
- net at C26.2: now also IC1_4.10, IC2_4.9 (B)
- removed net node_1: CP6., R108_1.1, R131.2, R98.2, R99.2
- net node_3: no longer names the net of R101.2, R127.2, R128.1
- net node_3: now also IC1_3.6 (B), IC1_4.9 (B)
- net node_4: no longer names the net of C25.1, Q16. (E)
- net node_4: now also IC2.1 (C)
- net node_5: no longer names the net of C25.2, Q19. (E)
- net node_5: now also IC2.5 (C)
- new net: C29.2, Q17. (E), Q18. (E)
- new net: C29.1, Q14. (E), Q15. (E)
- new net: IC1.2 (B), IC2_3.7
- new net: IC2_3.8 (C), IC2_4.11 (C)
- new net: IC1_5.12 (B), Q8. (E)
- new net: IC2_4.10, IC2_5.12 (B)
- new net: IC2.4 (B), R99.1
Other:
- note added: "CA3046"
- note added: "NAPOMENA 1 Kondenzatori koji moraju biti kvalitetni: C27,C29,C30,C71,C72,C73,C74,C75,C76,C77,C78"
- note removed: "IC1"
- note removed: "IC1_3"
- note removed: "IC1_4"
- note removed: "IC1_5"
- note removed: "IC2"
- note removed: "IC2_3"
- note removed: "IC2_4"
- note removed: "IC2_5"
- note removed: "NAPOMENA 1 Kondenzatori: C71,C72,C73,C74,C75,C76,C77,C78 su vrednosti 100n i oni su kvalitetniji"
- moved on the sheet: C25, C26, C27, C28, C29, C30, C71, C72, C73, C74, C75, C76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

Commit message: 08.07.2026 fix
Parts:
- removed R126_2: 2K, Resistor_THT:R_Axial_DIN0207_L6.3mm_D2.5mm_P7.62mm_Horizontal, symbol Device:R
- removed R128_1: 34K8, Resistor_THT:R_Axial_DIN0207_L6.3mm_D2.5mm_P7.62mm_Horizontal, symbol Device:R
- removed R128_2: 10K, Resistor_THT:R_Axial_DIN0207_L6.3mm_D2.5mm_P7.62mm_Horizontal, symbol Device:R
- C38: renamed from CP6; value 220u -> 220u/6V3
- R110: value 20K -> 20K 5%
- R126_1: value 49K -> 51K 5%
- R128_3: value 2K -> 36K 5%
- RV12: renamed from RV12_LIN; value 100K -> 100K LIN
- RV14: renamed from RV14_LOG; value 51K1 -> 51K1 LOG
- RV15: renamed from RV15_LIN; value 100K -> 100K LIN
- RV16: renamed from RV16_LOG; value 5K -> 5K LOG
- RV22: renamed from RV22_LIN; value 50K -> 50K LIN
- RV23: renamed from RV23_LIN; value 50K -> 50K LIN
- renumbered CP1 to C39, CP2 to C40
Connections:
- net -12V: now also R126_1.2, R128_3.1
- net enter_CP102 renamed Input ot C39
- new net: C29.2, Q17. (E), Q18. (E)
- new net: C29.1, Q14. (E), Q15. (E)
Other:
- note added: "PP"
- note removed: "NAPOMENA 1 Kondenzatori koji moraju biti kvalitetni: C27,C29,C30,C71,C72,C73,C74,C75,C76,C77,C78"
- moved on the sheet: R108_1, R126_1, R128_3

Commit message: Finalni deo seme, prelaz na PCB
Parts:
- renumbered C38 to C103, C39 to C104, C40 to C90
Connections:
- new net: C29.2, Q17. (E), Q18. (E)
- new net: C29.1, Q14. (E), Q15. (E)
Other:
- note added: "*GENERAL NOTE* Resistor values that are not explicitly specified are selected from the E96 value series with a tolerance of ±1%."
Changed lines of the file:
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@@
 		)
 	)
+	(text "*GENERAL NOTE*\nResistor values that are not explicitly specified\nare selected from the E96 value series with a \ntolerance of ±1%."
+		(exclude_from_sim no)
+		(at 299.974 247.396 0)
+		(effects
+			(font
+				(size 1.27 1.27)
+				(thickness 0.254)
+				(bold yes)
+			)
+			(justify left)
+		)
+	)
 	(junction
 		(at 270.51 128.27)
@@
 		(on_board yes)
 		(dnp no)
-		(property "Reference" "C39"
+		(property "Reference" "C104"
 			(at 78.994 180.086 0)
 			(effects
@@
 			(project "moog_prodigy_project"
 				(path "/db469bdb-b6c3-4a16-9199-d4e6b8d556e8/0831e821-0b52-4263-8fa0-a60bfb135571"
-					(reference "C39")
+					(reference "C104")
 					(unit 1)
 				)
@@
 		(on_board yes)
 		(dnp no)
-		(property "Reference" "C38"
+		(property "Reference" "C103"
 			(at 74.168 146.304 0)
 			(effects
@@
 			(project "moog_prodigy_project"
 				(path "/db469bdb-b6c3-4a16-9199-d4e6b8d556e8/0831e821-0b52-4263-8fa0-a60bfb135571"
-					(reference "C38")
+					(reference "C103")
 					(unit 1)
 				)
@@
 		(on_board yes)
 		(dnp no)
-		(property "Reference" "C40"
+		(property "Reference" "C90"
 			(at 159.766 142.494 90)
 			(effects
@@
 			(project "moog_prodigy_project"
 				(path "/db469bdb-b6c3-4a16-9199-d4e6b8d556e8/0831e821-0b52-4263-8fa0-a60bfb135571"
-					(reference "C40")
+					(reference "C90")
 					(unit 1)
 				)
